Commit message: Added f1

File: ffw_description/ros2_control/ffw_f1_follower/ffw_f1_follower.ros2_control.xacro (robot description, xacro)
@@ -1,6 +1,6 @@
 <?xml version="1.0"?>
 <robot xmlns:xacro="http://www.ros.org/wiki/xacro">
-  <xacro:macro name="ffw_f2_follower_system" params="use_sim:=^|false use_mock_hardware:=^|false mock_sensor_commands:=^|false">
-    <ros2_control name="ffw_f2_follower" type="system" is_async="true">
+  <xacro:macro name="ffw_f1_follower_system" params="use_sim:=^|false use_mock_hardware:=^|false mock_sensor_commands:=^|false">
+    <ros2_control name="ffw_f1_follower" type="system" is_async="true">
       <xacro:if value="$(arg use_sim)">
         <hardware>
@@ -20,6 +20,6 @@
             <param name="baud_rate">4000000</param>
             <param name="dynamixel_model_folder">/param/dxl_model</param>
-            <param name="number_of_joints">22</param>
-            <param name="number_of_transmissions">22</param>
+            <param name="number_of_joints">19</param>
+            <param name="number_of_transmissions">19</param>
             <param name="disable_torque_at_init">true</param>
             <param name="dynamixel_state_pub_msg_name">ffw_follower/dxl_state</param>
@@ -145,22 +145,4 @@
         <state_interface name="effort"/>
       </joint>
-      <joint name="left_wheel_steer">
-        <command_interface name="position"/>
-        <state_interface name="position"/>
-        <state_interface name="velocity"/>
-        <state_interface name="effort"/>
-      </joint>
-      <joint name="right_wheel_steer">
-        <command_interface name="position"/>
-        <state_interface name="position"/>
-        <state_interface name="velocity"/>
-        <state_interface name="effort"/>
-      </joint>
-      <joint name="rear_wheel_steer">
-        <command_interface name="position"/>
-        <state_interface name="position"/>
-        <state_interface name="velocity"/>
-        <state_interface name="effort"/>
-      </joint>
       <!-- RIGHT ARM -->
       <gpio name="dxl1">
@@ -172,5 +154,4 @@
         <state_interface name="Present Current"/>
         <state_interface name="Error Code"/>
-        <state_interface name="Present Input Voltage"/>
         <param name="Drive Mode">69</param>
         <param name="Operating Mode">3</param>
@@ -180,6 +161,6 @@
         <param name="Profile Velocity">3591</param>
         <param name="Profile Acceleration">3591</param>
-        <param name="Profile Acceleration Time">750</param>
-        <param name="Profile Time">1500</param>
+        <param name="Profile Acceleration Time">250</param>
+        <param name="Profile Time">500</param>
         <param name="Max Position Limit">262144</param>
         <param name="Min Position Limit">-262144</param>
@@ -204,6 +185,6 @@
         <param name="Profile Velocity">3591</param>
         <param name="Profile Acceleration">3591</param>
-        <param name="Profile Acceleration Time">750</param>
-        <param name="Profile Time">1500</param>
+        <param name="Profile Acceleration Time">250</param>
+        <param name="Profile Time">500</param>
         <param name="Max Position Limit">0</param>
         <param name="Min Position Limit">-262144</param>
@@ -228,6 +209,6 @@
         <param name="Profile Velocity">3591</param>
         <param name="Profile Acceleration">3591</param>
-        <param name="Profile Acceleration Time">750</param>
-        <param name="Profile Time">1500</param>
+        <param name="Profile Acceleration Time">250</param>
+        <param name="Profile Time">500</param>
         <param name="Max Position Limit">262144</param>
         <param name="Min Position Limit">-262144</param>
@@ -252,6 +233,6 @@
         <param name="Profile Velocity">6486</param>
         <param name="Profile Acceleration">3591</param>
-        <param name="Profile Acceleration Time">750</param>
-        <param name="Profile Time">1500</param>
+        <param name="Profile Acceleration Time">250</param>
+        <param name="Profile Time">500</param>
         <param name="Max Position Limit">90000</param>
         <param name="Min Position Limit">-245000</param>
@@ -276,6 +257,6 @@
         <param name="Profile Velocity">6486</param>
         <param name="Profile Acceleration">3591</param>
-        <param name="Profile Acceleration Time">750</param>
-        <param name="Profile Time">1500</param>
+        <param name="Profile Acceleration Time">250</param>
+        <param name="Profile Time">500</param>
         <param name="Max Position Limit">262144</param>
         <param name="Min Position Limit">-262144</param>
@@ -300,6 +281,6 @@
         <param name="Profile Velocity">6486</param>
         <param name="Profile Acceleration">3591</param>
-        <param name="Profile Acceleration Time">750</param>
-        <param name="Profile Time">1500</param>
+        <param name="Profile Acceleration Time">250</param>
+        <param name="Profile Time">500</param>
         <param name="Max Position Limit">131072</param>
         <param name="Min Position Limit">-131072</param>
@@ -323,6 +304,6 @@
         <param name="Acceleration Limit">359100</param>
         <param name="Current Limit">1500</param>
-        <param name="Profile Velocity">300</param>
-        <param name="Profile Acceleration">150</param>
+        <param name="Profile Velocity">100</param>
+        <param name="Profile Acceleration">50</param>
         <param name="Max Position Limit">131875</param>
         <param name="Min Position Limit">-151875</param>
@@ -357,6 +338,6 @@
         <param name="Profile Velocity">3591</param>
         <param name="Profile Acceleration">3591</param>
-        <param name="Profile Acceleration Time">750</param>
-        <param name="Profile Time">1500</param>
+        <param name="Profile Acceleration Time">250</param>
+        <param name="Profile Time">500</param>
         <param name="Max Position Limit">262144</param>
         <param name="Min Position Limit">-262144</param>
@@ -381,6 +362,6 @@
         <param name="Profile Velocity">3591</param>
         <param name="Profile Acceleration">3591</param>
-        <param name="Profile Acceleration Time">750</param>
-        <param name="Profile Time">1500</param>
+        <param name="Profile Acceleration Time">250</param>
+        <param name="Profile Time">500</param>
         <param name="Max Position Limit">262144</param>
         <param name="Min Position Limit">0</param>
@@ -405,6 +386,6 @@
         <param name="Profile Velocity">3591</param>
         <param name="Profile Acceleration">3591</param>
-        <param name="Profile Acceleration Time">750</param>
-        <param name="Profile Time">1500</param>
+        <param name="Profile Acceleration Time">250</param>
+        <param name="Profile Time">500</param>
         <param name="Max Position Limit">262144</param>
         <param name="Min Position Limit">-262144</param>
@@ -429,6 +410,6 @@
         <param name="Profile Velocity">6486</param>
         <param name="Profile Acceleration">3591</param>
-        <param name="Profile Acceleration Time">750</param>
-        <param name="Profile Time">1500</param>
+        <param name="Profile Acceleration Time">250</param>
+        <param name="Profile Time">500</param>
         <param name="Max Position Limit">90000</param>
         <param name="Min Position Limit">-245000</param>
@@ -453,6 +434,6 @@
         <param name="Profile Velocity">6486</param>
         <param name="Profile Acceleration">3591</param>
-        <param name="Profile Acceleration Time">750</param>
-        <param name="Profile Time">1500</param>
+        <param name="Profile Acceleration Time">250</param>
+        <param name="Profile Time">500</param>
         <param name="Max Position Limit">262144</param>
         <param name="Min Position Limit">-262144</param>
@@ -477,6 +458,6 @@
         <param name="Profile Velocity">6486</param>
         <param name="Profile Acceleration">3591</param>
-        <param name="Profile Acceleration Time">750</param>
-        <param name="Profile Time">1500</param>
+        <param name="Profile Acceleration Time">250</param>
+        <param name="Profile Time">500</param>
         <param name="Max Position Limit">131072</param>
         <param name="Min Position Limit">-131072</param>
@@ -500,6 +481,6 @@
         <param name="Acceleration Limit">359100</param>
         <param name="Current Limit">1500</param>
-        <param name="Profile Velocity">300</param>
-        <param name="Profile Acceleration">150</param>
+        <param name="Profile Velocity">100</param>
+        <param name="Profile Acceleration">50</param>
         <param name="Max Position Limit">131875</param>
         <param name="Min Position Limit">-151875</param>
@@ -534,6 +515,6 @@
         <param name="Profile Velocity">300</param>
         <param name="Profile Acceleration">300</param>
-        <param name="Profile Acceleration Time">750</param>
-        <param name="Profile Time">1500</param>
+        <param name="Profile Acceleration Time">250</param>
+        <param name="Profile Time">500</param>
         <param name="Max Position Limit">0</param>
         <param name="Min Position Limit">-50000</param>
@@ -557,11 +538,10 @@
         <state_interface name="Present Current"/>
         <state_interface name="Hardware Error Status"/>
-        <state_interface name="Present Input Voltage"/>
         <param name="Drive Mode">5</param>
         <param name="Operating Mode">3</param>
         <param name="Return Delay Time">0</param>
-        <param name="Profile Velocity">300</param>
-        <param name="Profile Acceleration">150</param>
-        <param name="Max Position Limit">2500</param>
+        <param name="Profile Velocity">100</param>
+        <param name="Profile Acceleration">50</param>
+        <param name="Max Position Limit">2560</param>
         <param name="Min Position Limit">1896</param>
         <param name="Position P Gain">1600</param>
@@ -582,6 +562,6 @@
         <param name="Operating Mode">3</param>
         <param name="Return Delay Time">0</param>
-        <param name="Profile Velocity">300</param>
-        <param name="Profile Acceleration">150</param>
+        <param name="Profile Velocity">100</param>
+        <param name="Profile Acceleration">50</param>
         <param name="Max Position Limit">2275</param>
         <param name="Min Position Limit">1820</param>
@@ -592,67 +572,4 @@
         <param name="Feedforward 2nd Gain">30</param>
       </gpio>
-      <!-- LEFT WHEEL -->
-      <gpio name="dxl101">
-        <param name="type">dxl</param>
-        <param name="ID">101</param>
-        <command_interface name="Goal Position"/>
-        <state_interface name="Present Position"/>
-        <state_interface name="Present Velocity"/>
-        <state_interface name="Present Current"/>
-        <state_interface name="Error Code"/>
-        <param name="Drive Mode">5</param>
-        <param name="Operating Mode">3</param>
-        <param name="Velocity Limit">12592</param>
-        <param name="Acceleration Limit">125920</param>
-        <param name="Min Position Limit">-1572864</param>
-        <param name="Max Position Limit">1572864</param>
-        <param name="Acceleration Limit">1010</param>
-        <param name="Return Delay Time">0</param>
-        <param name="Profile Velocity">12592</param>
-        <param name="Profile Acceleration Time">500</param>
-        <param name="Profile Time">1000</param>
-      </gpio>
-      <!-- RIGHT WHEEL -->
-      <gpio name="dxl103">
-        <param name="type">dxl</param>
-        <param name="ID">103</param>
-        <command_interface name="Goal Position"/>
-        <state_interface name="Present Position"/>
-        <state_interface name="Present Velocity"/>
-        <state_interface name="Present Current"/>
-        <state_interface name="Error Code"/>
-        <param name="Drive Mode">5</param>
-        <param name="Operating Mode">3</param>
-        <param name="Velocity Limit">12592</param>
-        <param name="Acceleration Limit">125920</param>
-        <param name="Min Position Limit">-1572864</param>
-        <param name="Max Position Limit">1572864</param>
-        <param name="Acceleration Limit">1010</param>
-        <param name="Return Delay Time">0</param>
-        <param name="Profile Velocity">12592</param>
-        <param name="Profile Acceleration Time">500</param>
-        <param name="Profile Time">1000</param>
-      </gpio>
-      <!-- REAR WHEEL -->
-      <gpio name="dxl105">
-        <param name="type">dxl</param>
-        <param name="ID">105</param>
-        <command_interface name="Goal Position"/>
-        <state_interface name="Present Position"/>
-        <state_interface name="Present Velocity"/>
-        <state_interface name="Present Current"/>
-        <state_interface name="Error Code"/>
-        <param name="Drive Mode">5</param>
-        <param name="Operating Mode">3</param>
-        <param name="Velocity Limit">12592</param>
-        <param name="Acceleration Limit">125920</param>
-        <param name="Min Position Limit">-1572864</param>
-        <param name="Max Position Limit">1572864</param>
-        <param name="Acceleration Limit">1010</param>
-        <param name="Return Delay Time">0</param>
-        <param name="Profile Velocity">12592</param>
-        <param name="Profile Acceleration Time">500</param>
-        <param name="Profile Time">1000</param>
-      </gpio>
     </ros2_control>
   </xacro:macro>

File: ffw_description/ros2_control/ffw_f1_follower/ffw_f1_follower_smooth.ros2_control.xacro (robot description, xacro)
@@ -1,6 +1,6 @@
 <?xml version="1.0"?>
 <robot xmlns:xacro="http://www.ros.org/wiki/xacro">
-  <xacro:macro name="ffw_f2_follower_system" params="use_sim:=^|false use_mock_hardware:=^|false mock_sensor_commands:=^|false">
-    <ros2_control name="ffw_f2_follower" type="system" is_async="true">
+  <xacro:macro name="ffw_f1_follower_system" params="use_sim:=^|false use_mock_hardware:=^|false mock_sensor_commands:=^|false">
+    <ros2_control name="ffw_f1_follower" type="system" is_async="true">
       <xacro:if value="$(arg use_sim)">
         <hardware>
@@ -20,11 +20,11 @@
             <param name="baud_rate">4000000</param>
             <param name="dynamixel_model_folder">/param/dxl_model</param>
-            <param name="number_of_joints">22</param>
-            <param name="number_of_transmissions">22</param>
+            <param name="number_of_joints">19</param>
+            <param name="number_of_transmissions">19</param>
             <param name="disable_torque_at_init">true</param>
-            <param name="dynamixel_state_pub_msg_name">ffw_follower/dxl_state</param>
-            <param name="get_dynamixel_data_srv_name">ffw_follower/get_dxl_data</param>
-            <param name="set_dynamixel_data_srv_name">ffw_follower/set_dxl_data</param>
-            <param name="reboot_dxl_srv_name">ffw_follower/reboot_dxl</param>
+            <param name="dynamixel_state_pub_msg_name">dynamixel_hardware_interface/dxl_state</param>
+            <param name="get_dynamixel_data_srv_name">dynamixel_hardware_interface/get_dxl_data</param>
+            <param name="set_dynamixel_data_srv_name">dynamixel_hardware_interface/set_dxl_data</param>
+            <param name="reboot_dxl_srv_name">dynamixel_hardware_interface/reboot_dxl</param>
             <param name="set_dxl_torque_srv_name">dynamixel_hardware_interface/set_dxl_torque</param>
           </xacro:unless>
@@ -145,22 +145,4 @@
         <state_interface name="effort"/>
       </joint>
-      <joint name="left_wheel_steer">
-        <command_interface name="position"/>
-        <state_interface name="position"/>
-        <state_interface name="velocity"/>
-        <state_interface name="effort"/>
-      </joint>
-      <joint name="right_wheel_steer">
-        <command_interface name="position"/>
-        <state_interface name="position"/>
-        <state_interface name="velocity"/>
-        <state_interface name="effort"/>
-      </joint>
-      <joint name="rear_wheel_steer">
-        <command_interface name="position"/>
-        <state_interface name="position"/>
-        <state_interface name="velocity"/>
-        <state_interface name="effort"/>
-      </joint>
       <!-- RIGHT ARM -->
       <gpio name="dxl1">
@@ -172,5 +154,4 @@
         <state_interface name="Present Current"/>
         <state_interface name="Error Code"/>
-        <state_interface name="Present Input Voltage"/>
         <param name="Drive Mode">69</param>
         <param name="Operating Mode">3</param>
@@ -557,5 +538,4 @@
         <state_interface name="Present Current"/>
         <state_interface name="Hardware Error Status"/>
-        <state_interface name="Present Input Voltage"/>
         <param name="Drive Mode">5</param>
         <param name="Operating Mode">3</param>
@@ -563,5 +543,5 @@
         <param name="Profile Velocity">300</param>
         <param name="Profile Acceleration">150</param>
-        <param name="Max Position Limit">2500</param>
+        <param name="Max Position Limit">2560</param>
         <param name="Min Position Limit">1896</param>
         <param name="Position P Gain">1600</param>
@@ -592,67 +572,4 @@
         <param name="Feedforward 2nd Gain">30</param>
       </gpio>
-      <!-- LEFT WHEEL -->
-      <gpio name="dxl101">
-        <param name="type">dxl</param>
-        <param name="ID">101</param>
-        <command_interface name="Goal Position"/>
-        <state_interface name="Present Position"/>
-        <state_interface name="Present Velocity"/>
-        <state_interface name="Present Current"/>
-        <state_interface name="Error Code"/>
-        <param name="Drive Mode">5</param>
-        <param name="Operating Mode">3</param>
-        <param name="Velocity Limit">12592</param>
-        <param name="Acceleration Limit">125920</param>
-        <param name="Min Position Limit">-1572864</param>
-        <param name="Max Position Limit">1572864</param>
-        <param name="Acceleration Limit">1010</param>
-        <param name="Return Delay Time">0</param>
-        <param name="Profile Velocity">12592</param>
-        <param name="Profile Acceleration Time">500</param>
-        <param name="Profile Time">1000</param>
-      </gpio>
-      <!-- RIGHT WHEEL -->
-      <gpio name="dxl103">
-        <param name="type">dxl</param>
-        <param name="ID">103</param>
-        <command_interface name="Goal Position"/>
-        <state_interface name="Present Position"/>
-        <state_interface name="Present Velocity"/>
-        <state_interface name="Present Current"/>
-        <state_interface name="Error Code"/>
-        <param name="Drive Mode">5</param>
-        <param name="Operating Mode">3</param>
-        <param name="Velocity Limit">12592</param>
-        <param name="Acceleration Limit">125920</param>
-        <param name="Min Position Limit">-1572864</param>
-        <param name="Max Position Limit">1572864</param>
-        <param name="Acceleration Limit">1010</param>
-        <param name="Return Delay Time">0</param>
-        <param name="Profile Velocity">12592</param>
-        <param name="Profile Acceleration Time">500</param>
-        <param name="Profile Time">1000</param>
-      </gpio>
-      <!-- REAR WHEEL -->
-      <gpio name="dxl105">
-        <param name="type">dxl</param>
-        <param name="ID">105</param>
-        <command_interface name="Goal Position"/>
-        <state_interface name="Present Position"/>
-        <state_interface name="Present Velocity"/>
-        <state_interface name="Present Current"/>
-        <state_interface name="Error Code"/>
-        <param name="Drive Mode">5</param>
-        <param name="Operating Mode">3</param>
-        <param name="Velocity Limit">12592</param>
-        <param name="Acceleration Limit">125920</param>
-        <param name="Min Position Limit">-1572864</param>
-        <param name="Max Position Limit">1572864</param>
-        <param name="Acceleration Limit">1010</param>
-        <param name="Return Delay Time">0</param>
-        <param name="Profile Velocity">12592</param>
-        <param name="Profile Acceleration Time">500</param>
-        <param name="Profile Time">1000</param>
-      </gpio>
     </ros2_control>
   </xacro:macro>

File: ffw_description/ros2_control/ffw_f2_follower/ffw_f2_follower.ros2_control.xacro (robot description, xacro)
@@ -317,5 +317,4 @@
         <state_interface name="Present Current"/>
         <state_interface name="Hardware Error Status"/>
-        <!-- <param name="Drive Mode">4</param> -->
         <param name="Drive Mode">5</param>
         <param name="Operating Mode">3</param>
@@ -495,5 +494,4 @@
         <state_interface name="Present Current"/>
         <state_interface name="Hardware Error Status"/>
-        <!-- <param name="Drive Mode">4</param> -->
         <param name="Drive Mode">5</param>
         <param name="Operating Mode">3</param>
