Commit message: Modified urdf and meshes for f1 and f2

File: ffw_description/gazebo/ffw_f1_follower/ffw_f1_follower.gazebo.xacro (robot description, xacro)
@@ -42,4 +42,5 @@
   <xacro:Link reference="arm_l_link6"/>
   <xacro:Link reference="arm_l_link7"/>
+  <!-- TODO: Change gripper to hx2_d1 -->
   <xacro:Link reference="r_rh_p12_rn_base"/>
   <xacro:Link reference="r_rh_p12_rn_r1"/>

File: ffw_description/gazebo/ffw_f2_follower/ffw_f2_follower.gazebo.xacro (robot description, xacro)
@@ -43,4 +43,5 @@
   <xacro:Link reference="arm_l_link6"/>
   <xacro:Link reference="arm_l_link7"/>
+  <!-- TODO: Change gripper to hx2_d1 -->
   <xacro:Link reference="r_rh_p12_rn_base"/>
   <xacro:Link reference="r_rh_p12_rn_r1"/>

File: ffw_description/urdf/common/follower/ffw_f_follower_body.xacro (robot description, xacro)
@@ -1,8 +1,8 @@
 <?xml version="1.0" encoding="UTF-8"?>
 <robot xmlns:xacro="http://www.ros.org/wiki/xacro">
-   <xacro:macro name="ffw_follower_body" params="prefix parent *origin">
+   <xacro:macro name="ffw_f_follower_body" params="prefix parent *origin">
       <xacro:include filename="$(find realsense2_description)/urdf/_d405.urdf.xacro" />
       <xacro:include filename="$(find ffw_description)/urdf/common/follower/zedm.urdf.xacro" />
-      <xacro:property name="meshes_file_direction" value="package://ffw_description/meshes/common/follower/ffw" />
+      <xacro:property name="meshes_file_direction" value="package://ffw_description/meshes/common/follower/ffw_f" />
       <joint name="${prefix}lift_joint" type="prismatic">
          <parent link="${parent}"/>
@@ -40,5 +40,5 @@
          <parent link="${prefix}arm_base_link" />
          <child link="${prefix}head_link1" />
-         <origin xyz="0.049483 0 0.102130" rpy="0 0 0" />
+         <origin xyz="0.102729 0 0.132803" rpy="0 0 0" />
          <axis xyz="0 1 0" />
          <limit velocity="4.8" effort="1000" lower="-0.2317" upper="0.6951" />
@@ -72,5 +72,5 @@
          <parent link="${prefix}head_link1" />
          <child link="${prefix}head_link2" />
-         <origin xyz="0.040 0 0.054" rpy="0 0 0" />
+         <origin xyz="0.0141410 0 0.0555070" rpy="0 0 0" />
          <axis xyz="0 0 1" />
          <limit velocity="4.8" effort="1000" lower="-0.35" upper="0.35" />
@@ -110,5 +110,5 @@
          <parent link="${prefix}arm_base_link" />
          <child link="${prefix}arm_l_link1" />
-         <origin xyz="0 0.1045 0" rpy="0 0 0" />
+         <origin xyz="0.059 0.1127 0.030" rpy="0 0 0" />
          <axis xyz="0 1 0" />
          <limit velocity="4.8" effort="1000" lower="-3.14" upper="3.14" />
@@ -142,5 +142,5 @@
          <parent link="${prefix}arm_l_link1" />
          <child link="${prefix}arm_l_link2" />
-         <origin xyz="0 0.123 0" rpy="0 0 0" />
+         <origin xyz="0.0177 0.1038 0" rpy="0 0 0" />
          <axis xyz="1 0 0" />
          <limit velocity="4.8" effort="1000" lower="0.0" upper="3.14" />
@@ -174,5 +174,5 @@
          <parent link="${prefix}arm_l_link2" />
          <child link="${prefix}arm_l_link3" />
-         <origin xyz="0 0 -0.165" rpy="0 0 0" />
+         <origin xyz="-0.0177 0 -0.2072" rpy="0 0 0" />
          <axis xyz="0 0 1" />
          <limit velocity="4.8" effort="1000" lower="-3.14" upper="3.14" />
@@ -206,5 +206,5 @@
          <parent link="${prefix}arm_l_link3" />
          <child link="${prefix}arm_l_link4" />
-         <origin xyz="0.041004 0 -0.135" rpy="0 0 0" />
+         <origin xyz="0.0410041 0.0007 -0.1128" rpy="0 0 0" />
          <axis xyz="0 1 0" />
          <limit velocity="4.8" effort="1000" lower="-2.9361" upper="1.0786" />
@@ -238,5 +238,5 @@
          <parent link="${prefix}arm_l_link4" />
          <child link="${prefix}arm_l_link5" />
-         <origin xyz="-0.041004 0 -0.1489" rpy="0 0 0" />
+         <origin xyz="-0.041 -0.0007 -0.1477" rpy="0 0 0" />
          <axis xyz="0 0 1" />
          <limit velocity="4.8" effort="1000" lower="-3.14" upper="3.14" />
@@ -270,5 +270,5 @@
          <parent link="${prefix}arm_l_link5" />
          <child link="${prefix}arm_l_link6" />
-         <origin xyz="0 0 -0.1041" rpy="0 0 0" />
+         <origin xyz="0 0.0007 -0.0948" rpy="0 0 0" />
          <axis xyz="0 1 0" />
          <limit velocity="4.8" effort="1000" lower="-1.57" upper="1.57" />
@@ -302,5 +302,5 @@
          <parent link="${prefix}arm_l_link6" />
          <child link="${prefix}arm_l_link7" />
-         <origin xyz="0 0 -0.0885" rpy="0 0 0" />
+         <origin xyz="0 -0.0007 -0.0775" rpy="0 0 0" />
          <axis xyz="1 0 0" />
          <limit velocity="4.8" effort="1000" lower="-1.8201" upper="1.5804" />
@@ -337,5 +337,5 @@
          <parent link="${prefix}arm_base_link" />
          <child link="${prefix}arm_r_link1" />
-         <origin xyz="0 -0.1045 0" rpy="0 0 0" />
+         <origin xyz="0.055 -0.1127 0.030" rpy="0 0 0" />
          <axis xyz="0 1 0" />
          <limit velocity="4.8" effort="1000" lower="-3.14" upper="3.14" />
@@ -369,5 +369,5 @@
          <parent link="${prefix}arm_r_link1" />
          <child link="${prefix}arm_r_link2" />
-         <origin xyz="0 -0.123 0" rpy="0 0 0" />
+         <origin xyz="0.0177 -0.1038 0" rpy="0 0 0" />
          <axis xyz="1 0 0" />
          <limit velocity="4.8" effort="1000" lower="-3.14" upper="0" />
@@ -401,5 +401,5 @@
          <parent link="${prefix}arm_r_link2" />
          <child link="${prefix}arm_r_link3" />
-         <origin xyz="0 0 -0.165" rpy="0 0 0" />
+         <origin xyz="-0.0177 0 -0.2072" rpy="0 0 0" />
          <axis xyz="0 0 1" />
          <limit velocity="4.8" effort="1000" lower="-3.14" upper="3.14" />
@@ -433,5 +433,5 @@
          <parent link="${prefix}arm_r_link3" />
          <child link="${prefix}arm_r_link4" />
-         <origin xyz="0.041004 0 -0.135" rpy="0 0 0" />
+         <origin xyz="0.0410041 -0.0007 -0.1128" rpy="0 0 0" />
          <axis xyz="0 1 0" />
          <limit velocity="4.8" effort="1000" lower="-2.9361" upper="1.0786" />
@@ -465,5 +465,5 @@
          <parent link="${prefix}arm_r_link4" />
          <child link="${prefix}arm_r_link5" />
-         <origin xyz="-0.041004 0 -0.1489" rpy="0 0 0" />
+         <origin xyz="-0.041 0.0007 -0.1477" rpy="0 0 0" />
          <axis xyz="0 0 1" />
          <limit velocity="4.8" effort="1000" lower="-3.14" upper="3.14" />
@@ -497,5 +497,5 @@
          <parent link="${prefix}arm_r_link5" />
          <child link="${prefix}arm_r_link6" />
-         <origin xyz="0 0 -0.1041" rpy="0 0 0" />
+         <origin xyz="0 -0.0007 -0.0948" rpy="0 0 0" />
          <axis xyz="0 1 0" />
          <limit velocity="4.8" effort="1000" lower="-1.57" upper="1.57" />
@@ -529,5 +529,5 @@
          <parent link="${prefix}arm_r_link6" />
          <child link="${prefix}arm_r_link7" />
-         <origin xyz="0 0 -0.0885" rpy="0 0 0" />
+         <origin xyz="-0.00025 -0.0007 -0.0775" rpy="0 0 0" />
          <axis xyz="1 0 0" />
          <limit velocity="4.8" effort="1000" lower="-1.5804" upper="1.8201" />

File: ffw_description/urdf/ffw_f1_follower/ffw_f1_follower.urdf.xacro (robot description, xacro)
@@ -9,5 +9,6 @@
   <xacro:arg name="model" default="ffw_f1_follower" />
   <xacro:arg name="ros2_control_type" default="ffw_f1_follower" />
-  <xacro:include filename="$(find ffw_description)/urdf/common/follower/ffw_follower_body.xacro" />
+  <xacro:include filename="$(find ffw_description)/urdf/common/follower/ffw_f_follower_body.xacro" />
+  <!-- TODO: Change gripper to hx2_d1 -->
   <xacro:include filename="$(find ffw_description)/urdf/common/rh_p12_rn_a/rh_p12_rn_a.urdf.xacro" />
   <xacro:include filename="$(find ffw_description)/ros2_control/$(arg model)/$(arg ros2_control_type).ros2_control.xacro" />
@@ -43,7 +44,8 @@
     </inertial>
   </link>
-  <xacro:ffw_follower_body parent="$(arg prefix)base_link" prefix="$(arg prefix)">
+  <xacro:ffw_f_follower_body parent="$(arg prefix)base_link" prefix="$(arg prefix)">
     <origin xyz="0.0055 0 1.4316" rpy="0 0 0" />
-  </xacro:ffw_follower_body>
+  </xacro:ffw_f_follower_body>
+  <!-- TODO: Change gripper to hx2_d1 -->
   <xacro:rh_p12_rn_a parent="$(arg prefix)arm_l_link7" prefix="$(arg prefix)gripper_l_">
     <origin xyz="0 0 -0.078" rpy="0 3.14159265359 3.14159265359"/>
@@ -65,4 +67,5 @@
     </visual>
   </link>
+  <!-- TODO: Change gripper to hx2_d1 -->
   <xacro:rh_p12_rn_a parent="$(arg prefix)arm_r_link7" prefix="$(arg prefix)gripper_r_">
     <origin xyz="0 0 -0.078" rpy="0 3.14159265359 3.14159265359"/>

File: ffw_description/urdf/ffw_f2_follower/ffw_f2_follower.urdf.xacro (robot description, xacro)
@@ -9,5 +9,6 @@
   <xacro:arg name="model" default="ffw_f2_follower" />
   <xacro:arg name="ros2_control_type" default="ffw_f2_follower" />
-  <xacro:include filename="$(find ffw_description)/urdf/common/follower/ffw_follower_body.xacro" />
+  <xacro:include filename="$(find ffw_description)/urdf/common/follower/ffw_f_follower_body.xacro" />
+  <!-- TODO: Change gripper to hx2_d1 -->
   <xacro:include filename="$(find ffw_description)/urdf/common/rh_p12_rn_a/rh_p12_rn_a.urdf.xacro" />
   <xacro:include filename="$(find ffw_description)/ros2_control/$(arg model)/$(arg ros2_control_type).ros2_control.xacro" />
@@ -114,7 +115,8 @@
   <!-- Gazebo plugins/sensors -->
   <xacro:ffw_f2_follower_gazebo prefix="$(arg prefix)" />
-  <xacro:ffw_follower_body parent="$(arg prefix)base_link" prefix="$(arg prefix)">
+  <xacro:ffw_f_follower_body parent="$(arg prefix)base_link" prefix="$(arg prefix)">
     <origin xyz="-0.0199 0 1.4316" rpy="0 0 0" />
-  </xacro:ffw_follower_body>
+  </xacro:ffw_f_follower_body>
+  <!-- TODO: Change gripper to hx2_d1 -->
   <xacro:rh_p12_rn_a parent="$(arg prefix)arm_l_link7" prefix="$(arg prefix)gripper_l_">
     <origin xyz="0 0 -0.078" rpy="0 3.14159265359 3.14159265359"/>
@@ -136,4 +138,5 @@
     </visual>
   </link>
+  <!-- TODO: Change gripper to hx2_d1 -->
   <xacro:rh_p12_rn_a parent="$(arg prefix)arm_r_link7" prefix="$(arg prefix)gripper_r_">
     <origin xyz="0 0 -0.078" rpy="0 3.14159265359 3.14159265359"/>
