Commit message: Added base meshes

File: ffw_description/urdf/ffw_bg2_rev4_follower/ffw_bg2_follower.urdf.xacro (robot description, xacro)
@@ -2,5 +2,5 @@
 <robot xmlns:xacro="http://www.ros.org/wiki/xacro" name="ffw_bg2_follower">
   <xacro:property name="meshes_file_direction" value="package://ffw_description/meshes/$(arg model)" />
-  <xacro:property name="base_meshes_dir" value="package://ffw_description/meshes/common/follower/base" />
+  <xacro:property name="base_meshes_dir" value="package://ffw_description/meshes/common/follower/ffw_base" />
   <xacro:arg name="use_sim" default="false" />
   <xacro:arg name="use_mock_hardware" default="false" />

File: ffw_description/urdf/ffw_bh5_rev1_follower/ffw_bh5_follower.urdf.xacro (robot description, xacro)
@@ -2,5 +2,5 @@
 <robot xmlns:xacro="http://www.ros.org/wiki/xacro" name="ffw_bh5_follower">
   <xacro:property name="meshes_file_direction" value="package://ffw_description/meshes/$(arg model)" />
-  <xacro:property name="base_meshes_dir" value="package://ffw_description/meshes/common/follower/base" />
+  <xacro:property name="base_meshes_dir" value="package://ffw_description/meshes/common/follower/ffw_base" />
   <xacro:arg name="use_sim" default="false" />
   <xacro:arg name="use_mock_hardware" default="false" />

File: ffw_description/urdf/ffw_f1_follower/ffw_f1_follower.urdf.xacro (robot description, xacro)
@@ -2,5 +2,5 @@
 <robot xmlns:xacro="http://www.ros.org/wiki/xacro" name="ffw_f1_follower">
   <xacro:property name="meshes_file_direction" value="package://ffw_description/meshes/$(arg model)" />
-  <xacro:property name="base_meshes_dir" value="package://ffw_description/meshes/common/follower/base" />
+  <xacro:property name="base_meshes_dir" value="package://ffw_description/meshes/common/follower/ffw_f_base" />
   <xacro:arg name="use_sim" default="false" />
   <xacro:arg name="use_mock_hardware" default="false" />

File: ffw_description/urdf/ffw_f2_follower/ffw_f2_follower.urdf.xacro (robot description, xacro)
@@ -2,5 +2,5 @@
 <robot xmlns:xacro="http://www.ros.org/wiki/xacro" name="ffw_f2_follower">
   <xacro:property name="meshes_file_direction" value="package://ffw_description/meshes/$(arg model)" />
-  <xacro:property name="swerve_meshes_dir" value="package://ffw_description/meshes/common/follower/swerve" />
+  <xacro:property name="swerve_meshes_dir" value="package://ffw_description/meshes/common/follower/ffw_f_swerve" />
   <xacro:arg name="use_sim" default="false" />
   <xacro:arg name="use_mock_hardware" default="false" />
@@ -44,5 +44,5 @@
     <parent link="$(arg prefix)base_link"/>
     <child link="$(arg prefix)lidar_l_link"/>
-    <origin xyz="-0.111881 0.240 0.34432" rpy="0 0 1.57079632679"/>
+    <origin xyz="-0.111881 0.240 0.35015" rpy="0 0 1.57079632679"/>
   </joint>
   <link name="$(arg prefix)lidar_l_link">
@@ -60,5 +60,5 @@
     <parent link="$(arg prefix)base_link"/>
     <child link="$(arg prefix)lidar_r_link"/>
-    <origin xyz="-0.111881 -0.240 0.34432" rpy="0 0 -1.57079632679"/>
+    <origin xyz="-0.111881 -0.240 0.35015" rpy="0 0 -1.57079632679"/>
   </joint>
   <!-- <link name="$(arg prefix)lidar_r_link">
@@ -67,5 +67,5 @@
     <parent link="$(arg prefix)base_link"/>
     <child link="$(arg prefix)imu_link"/>
-    <origin xyz="-0.1464 0.0 0.26" rpy="0 0 0"/>
+    <origin xyz="-0.189181 0.0 0.247" rpy="0 0 0"/>
   </joint>
   <link name="$(arg prefix)imu_link">
@@ -116,5 +116,5 @@
   <xacro:ffw_f2_follower_gazebo prefix="$(arg prefix)" />
   <xacro:ffw_f_follower_body parent="$(arg prefix)base_link" prefix="$(arg prefix)">
-    <origin xyz="-0.0199 0 1.4316" rpy="0 0 0" />
+    <origin xyz="-0.0753807 0 1.407" rpy="0 0 0" />
   </xacro:ffw_f_follower_body>
   <!-- TODO: Change gripper to hx2_d1 -->
@@ -161,5 +161,5 @@
       <parent link="$(arg prefix)base_link"/>
       <child link="$(arg prefix)left_wheel_steer_link"/>
-      <origin xyz="0.1371 0.2554 0.27555" rpy="0 0 0"/>
+      <origin xyz="0.137119 0.2554 0.2613" rpy="0 0 0"/>
       <axis xyz="0 0 1" />
       <limit velocity="9999.0" effort="9999.0" lower="${-pi*6.0}" upper="${pi*6.0}" />
@@ -192,5 +192,5 @@
       <parent link="$(arg prefix)left_wheel_steer_link"/>
       <child link="$(arg prefix)left_wheel_drive_link"/>
-      <origin xyz="0 0 -0.18905" rpy="0 0 0"/>
+      <origin xyz="0 0 -0.1748" rpy="0 0 0"/>
       <axis xyz="0 1 0" />
       <limit velocity="9999.0" effort="9999.0"/>
@@ -229,5 +229,5 @@
       <parent link="$(arg prefix)base_link"/>
       <child link="$(arg prefix)right_wheel_steer_link"/>
-      <origin xyz="0.1371 -0.2554 0.27555" rpy="0 0 0"/>
+      <origin xyz="0.137119 -0.2554 0.2613" rpy="0 0 0"/>
       <axis xyz="0 0 1" />
       <limit velocity="9999.0" effort="9999.0" lower="${-pi*6.0}" upper="${pi*6.0}" />
@@ -260,5 +260,5 @@
       <parent link="$(arg prefix)right_wheel_steer_link"/>
       <child link="$(arg prefix)right_wheel_drive_link"/>
-      <origin xyz="0 0 -0.18905" rpy="0 0 0"/>
+      <origin xyz="0 0 -0.1748" rpy="0 0 0"/>
       <axis xyz="0 1 0" />
       <limit velocity="9999.0" effort="9999.0"/>
@@ -297,5 +297,5 @@
       <parent link="$(arg prefix)base_link"/>
       <child link="$(arg prefix)rear_wheel_steer_link"/>
-      <origin xyz="-0.2899 0 0.27555" rpy="0 0 0"/>
+      <origin xyz="-0.288133 0 0.2613" rpy="0 0 0"/>
       <axis xyz="0 0 1" />
       <limit velocity="9999.0" effort="9999.0" lower="${-pi*6.0}" upper="${pi*6.0}" />
@@ -328,5 +328,5 @@
       <parent link="$(arg prefix)rear_wheel_steer_link"/>
       <child link="$(arg prefix)rear_wheel_drive_link"/>
-      <origin xyz="0 0 -0.18905" rpy="0 0 0"/>
+      <origin xyz="0 0 -0.1748" rpy="0 0 0"/>
       <axis xyz="0 1 0" />
       <limit velocity="9999.0" effort="9999.0"/>

File: ffw_description/urdf/ffw_sg2_rev1_follower/ffw_sg2_follower.urdf.xacro (robot description, xacro)
@@ -2,5 +2,5 @@
 <robot xmlns:xacro="http://www.ros.org/wiki/xacro" name="ffw_sg2_follower">
   <xacro:property name="meshes_file_direction" value="package://ffw_description/meshes/$(arg model)" />
-  <xacro:property name="swerve_meshes_dir" value="package://ffw_description/meshes/common/follower/swerve" />
+  <xacro:property name="swerve_meshes_dir" value="package://ffw_description/meshes/common/follower/ffw_swerve" />
   <xacro:arg name="use_sim" default="false" />
   <xacro:arg name="use_mock_hardware" default="false" />

File: ffw_description/urdf/ffw_sh5_rev1_follower/ffw_sh5_follower.urdf.xacro (robot description, xacro)
@@ -2,5 +2,5 @@
 <robot xmlns:xacro="http://www.ros.org/wiki/xacro" name="ffw_sh5_follower">
   <xacro:property name="meshes_file_direction" value="package://ffw_description/meshes/$(arg model)" />
-  <xacro:property name="swerve_meshes_dir" value="package://ffw_description/meshes/common/follower/swerve" />
+  <xacro:property name="swerve_meshes_dir" value="package://ffw_description/meshes/common/follower/ffw_swerve" />
   <xacro:arg name="use_sim" default="false" />
   <xacro:arg name="use_mock_hardware" default="false" />
