Commit message: Modified urdf mesh file paths

File: ffw_description/urdf/ffw_bg2_rev4_follower/ffw_bg2_follower.urdf (robot description, URDF)
Before this commit: robot ffw_bg2_follower, 41 links, 40 joints
Links:
- link zedm_camera_center: geometry collision mesh filename=package://ffw_description/meshes/common/follower/zedm.stl scale=0.001 0.001 0.001; visual mesh filename=package://ffw_description/meshes/common/follower/zedm.stl scale=0.001 0.001 0.001

File: ffw_description/urdf/ffw_f1_follower/ffw_f1_follower.urdf (robot description, URDF)
Before this commit: robot ffw_f1_follower, 37 links, 36 joints
Links:
- link camera_l_base_link: geometry collision mesh filename=package://ffw_description/meshes/common/follower/wrist_d401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 scale=0.001 0.001 0.001; visual mesh filename=package://ffw_description/meshes/common/follower/wrist_d401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 scale=0.001 0.001 0.001
- link camera_r_base_link: geometry collision mesh filename=package://ffw_description/meshes/common/follower/wrist_d401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 scale=0.001 0.001 0.001; visual mesh filename=package://ffw_description/meshes/common/follower/wrist_d401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 scale=0.001 0.001 0.001

File: ffw_description/urdf/ffw_f2_follower/ffw_f2_follower.urdf (robot description, URDF)
Before this commit: robot ffw_f2_follower, 46 links, 45 joints
Links:
- link camera_l_base_link: geometry collision mesh filename=package://ffw_description/meshes/common/follower/wrist_d401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 scale=0.001 0.001 0.001; visual mesh filename=package://ffw_description/meshes/common/follower/wrist_d401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 scale=0.001 0.001 0.001
- link camera_r_base_link: geometry collision mesh filename=package://ffw_description/meshes/common/follower/wrist_d401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 scale=0.001 0.001 0.001; visual mesh filename=package://ffw_description/meshes/common/follower/wrist_d401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 scale=0.001 0.001 0.001

File: ffw_description/urdf/ffw_sg2_rev1_follower/ffw_sg2_follower.urdf (robot description, URDF)
Before this commit: robot ffw_sg2_follower, 50 links, 49 joints
Links:
- link zedm_camera_center: geometry collision mesh filename=package://ffw_description/meshes/common/follower/zedm.stl scale=0.001 0.001 0.001; visual mesh filename=package://ffw_description/meshes/common/follower/zedm.stl scale=0.001 0.001 0.001

File: ffw_description/urdf/ffw_sh5_rev1_follower/ffw_sh5_follower.urdf (robot description, URDF)
Before this commit: robot ffw_sh5_follower, 92 links, 91 joints
Links:
- link zedm_camera_center: geometry collision mesh filename=package://ffw_description/meshes/common/follower/zedm.stl scale=0.001 0.001 0.001; visual mesh filename=package://ffw_description/meshes/common/follower/zedm.stl scale=0.001 0.001 0.001

Commit message: Update link names

File: ffw_description/urdf/ffw_bg2_rev4_follower/ffw_bg2_follower.urdf (robot description, URDF)
Before this commit: robot ffw_bg2_follower, 41 links, 40 joints
Links:
- removed link camera_l_bottom_screw_frame
- removed link camera_l_link
- removed link camera_r_bottom_screw_frame
- removed link camera_r_link
- removed link zedm_camera_center
- removed link zedm_camera_link
- removed link zedm_left_camera_frame
- removed link zedm_left_camera_optical_frame
- removed link zedm_right_camera_frame
- removed link zedm_right_camera_optical_frame
- added link camera_left_bottom_screw_frame
- added link camera_left_link, mass 0.072; collision box size=0.023 0.042 0.042; visual mesh filename=file:///root/ros2_ws/install/realsense2_description/share/r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 scale=0.001 0.001 0.001
- added link camera_right_bottom_screw_frame
- added link camera_right_link, mass 0.072; collision box size=0.023 0.042 0.042; visual mesh filename=file:///root/ros2_ws/install/realsense2_description/share/r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 scale=0.001 0.001 0.001
- added link zed_camera_center; collision mesh filename=package://ffw_description/meshes/common/follower/zedm.stl scale=0.001 0.001 0.001; visual mesh filename=package://ffw_description/meshes/common/follower/zedm.stl scale=0.001 0.001 0.001
- added link zed_camera_link
- added link zed_left_camera_frame
- added link zed_left_camera_optical_frame
- added link zed_right_camera_frame
- added link zed_right_camera_optical_frame
Joints:
- removed joint camera_l_joint
- removed joint camera_l_link_joint
- removed joint camera_r_joint
- removed joint camera_r_link_joint
- removed joint zedm_camera_center_joint
- removed joint zedm_joint
- removed joint zedm_left_camera_joint
- removed joint zedm_left_camera_optical_joint
- removed joint zedm_right_camera_joint
- removed joint zedm_right_camera_optical_joint
- added joint camera_left_joint: type fixed, parent arm_l_link7, child camera_left_bottom_screw_frame, origin xyz=0.108236 -0.021 -0.062552 rpy=-1.57079632679 1.66678943569 0
- added joint camera_left_link_joint: type fixed, parent camera_left_bottom_screw_frame, child camera_left_link, origin xyz=0.01085 0.009 0.021 rpy=0 0 0
- added joint camera_right_joint: type fixed, parent arm_r_link7, child camera_right_bottom_screw_frame, origin xyz=0.108236 -0.021 -0.062552 rpy=-1.57079632679 1.66678943569 0
- added joint camera_right_link_joint: type fixed, parent camera_right_bottom_screw_frame, child camera_right_link, origin xyz=0.01085 0.009 0.021 rpy=0 0 0
- added joint zed_camera_center_joint: type fixed, parent zed_camera_link, child zed_camera_center, origin xyz=0 0 0.01325 rpy=0 0 0
- added joint zed_joint: type fixed, parent head_link2, child zed_camera_link, origin xyz=0.0238122 -0.00651797 -0.0242094 rpy=0 0 0
- added joint zed_left_camera_joint: type fixed, parent zed_camera_center, child zed_left_camera_frame, origin xyz=0 0.0315 0 rpy=0 0 0
- added joint zed_left_camera_optical_joint: type fixed, parent zed_left_camera_frame, child zed_left_camera_optical_frame, origin xyz=0 0 0 rpy=-1.57079632679 0.0 -1.57079632679
- added joint zed_right_camera_joint: type fixed, parent zed_camera_center, child zed_right_camera_frame, origin xyz=0 -0.0315 0 rpy=0 0 0
- added joint zed_right_camera_optical_joint: type fixed, parent zed_right_camera_frame, child zed_right_camera_optical_frame, origin xyz=0 0 0 rpy=-1.57079632679 0.0 -1.57079632679

File: ffw_description/urdf/ffw_f1_follower/ffw_f1_follower.urdf (robot description, URDF)
Before this commit: robot ffw_f1_follower, 37 links, 36 joints
Links:
- removed link camera_l_base_link
- removed link camera_l_link
- removed link camera_r_base_link
- removed link camera_r_link
- added link camera_left_base_link, mass 3.6935029e-02; collision mesh filename=package://ffw_description/meshes/common/follower/wrist_d401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 scale=0.001 0.001 0.001; visual mesh filename=package://ffw_description/meshes/common/follower/wrist_d401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 scale=0.001 0.001 0.001
- added link camera_left_link
- added link camera_right_base_link, mass 3.6935029e-02; collision mesh filename=package://ffw_description/meshes/common/follower/wrist_d401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 scale=0.001 0.001 0.001; visual mesh filename=package://ffw_description/meshes/common/follower/wrist_d401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 scale=0.001 0.001 0.001
- added link camera_right_link
Joints:
- removed joint camera_l_joint
- removed joint camera_l_link_joint
- removed joint camera_r_joint
- removed joint camera_r_link_joint
- added joint camera_left_joint: type fixed, parent camera_left_base_link, child camera_left_link, origin xyz=0.0126724 -0.02235 0.009 rpy=0 0 0.3490656
- added joint camera_left_link_joint: type fixed, parent arm_l_link7, child camera_left_base_link, origin xyz=0.0275 0.0 -0.0847501 rpy=-1.57079632679 1.57079632679 0
- added joint camera_right_joint: type fixed, parent camera_right_base_link, child camera_right_link, origin xyz=0.0126724 -0.02235 0.009 rpy=0 0 0.3490656
- added joint camera_right_link_joint: type fixed, parent arm_r_link7, child camera_right_base_link, origin xyz=0.0275 0.0 -0.0847501 rpy=-1.57079632679 1.57079632679 0

File: ffw_description/urdf/ffw_f2_follower/ffw_f2_follower.urdf (robot description, URDF)
Before this commit: robot ffw_f2_follower, 46 links, 45 joints
Links:
- removed link camera_l_base_link
- removed link camera_l_link
- removed link camera_r_base_link
- removed link camera_r_link
- added link camera_left_base_link, mass 3.6935029e-02; collision mesh filename=package://ffw_description/meshes/common/follower/wrist_d401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 scale=0.001 0.001 0.001; visual mesh filename=package://ffw_description/meshes/common/follower/wrist_d401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 scale=0.001 0.001 0.001
- added link camera_left_link
- added link camera_right_base_link, mass 3.6935029e-02; collision mesh filename=package://ffw_description/meshes/common/follower/wrist_d401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 scale=0.001 0.001 0.001; visual mesh filename=package://ffw_description/meshes/common/follower/wrist_d401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 scale=0.001 0.001 0.001
- added link camera_right_link
Joints:
- removed joint camera_l_joint
- removed joint camera_l_link_joint
- removed joint camera_r_joint
- removed joint camera_r_link_joint
- added joint camera_left_joint: type fixed, parent camera_left_base_link, child camera_left_link, origin xyz=0.0126724 -0.02235 0.009 rpy=0 0 0.3490656
- added joint camera_left_link_joint: type fixed, parent arm_l_link7, child camera_left_base_link, origin xyz=0.0275 0.0 -0.0847501 rpy=-1.57079632679 1.57079632679 0
- added joint camera_right_joint: type fixed, parent camera_right_base_link, child camera_right_link, origin xyz=0.0126724 -0.02235 0.009 rpy=0 0 0.3490656
- added joint camera_right_link_joint: type fixed, parent arm_r_link7, child camera_right_base_link, origin xyz=0.0275 0.0 -0.0847501 rpy=-1.57079632679 1.57079632679 0

File: ffw_description/urdf/ffw_sg2_rev1_follower/ffw_sg2_follower.urdf (robot description, URDF)
Before this commit: robot ffw_sg2_follower, 50 links, 49 joints
Links:
- removed link camera_l_bottom_screw_frame
- removed link camera_l_link
- removed link camera_r_bottom_screw_frame
- removed link camera_r_link
- removed link zedm_camera_center
- removed link zedm_camera_link
- removed link zedm_left_camera_frame
- removed link zedm_left_camera_optical_frame
- removed link zedm_right_camera_frame
- removed link zedm_right_camera_optical_frame
- added link camera_left_bottom_screw_frame
- added link camera_left_link, mass 0.072; collision box size=0.023 0.042 0.042; visual mesh filename=file:///root/ros2_ws/install/realsense2_description/share/r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 scale=0.001 0.001 0.001
- added link camera_right_bottom_screw_frame
- added link camera_right_link, mass 0.072; collision box size=0.023 0.042 0.042; visual mesh filename=file:///root/ros2_ws/install/realsense2_description/share/r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 scale=0.001 0.001 0.001
- added link zed_camera_center; collision mesh filename=package://ffw_description/meshes/common/follower/zedm.stl scale=0.001 0.001 0.001; visual mesh filename=package://ffw_description/meshes/common/follower/zedm.stl scale=0.001 0.001 0.001
- added link zed_camera_link
- added link zed_left_camera_frame
- added link zed_left_camera_optical_frame
- added link zed_right_camera_frame
- added link zed_right_camera_optical_frame
Joints:
- removed joint camera_l_joint
- removed joint camera_l_link_joint
- removed joint camera_r_joint
- removed joint camera_r_link_joint
- removed joint zedm_camera_center_joint
- removed joint zedm_joint
- removed joint zedm_left_camera_joint
- removed joint zedm_left_camera_optical_joint
- removed joint zedm_right_camera_joint
- removed joint zedm_right_camera_optical_joint
- added joint camera_left_joint: type fixed, parent arm_l_link7, child camera_left_bottom_screw_frame, origin xyz=0.108236 -0.021 -0.062552 rpy=-1.57079632679 1.66678943569 0
- added joint camera_left_link_joint: type fixed, parent camera_left_bottom_screw_frame, child camera_left_link, origin xyz=0.01085 0.009 0.021 rpy=0 0 0
- added joint camera_right_joint: type fixed, parent arm_r_link7, child camera_right_bottom_screw_frame, origin xyz=0.108236 -0.021 -0.062552 rpy=-1.57079632679 1.66678943569 0
- added joint camera_right_link_joint: type fixed, parent camera_right_bottom_screw_frame, child camera_right_link, origin xyz=0.01085 0.009 0.021 rpy=0 0 0
- added joint zed_camera_center_joint: type fixed, parent zed_camera_link, child zed_camera_center, origin xyz=0 0 0.01325 rpy=0 0 0
- added joint zed_joint: type fixed, parent head_link2, child zed_camera_link, origin xyz=0.0238122 -0.00651797 -0.0242094 rpy=0 0 0
- added joint zed_left_camera_joint: type fixed, parent zed_camera_center, child zed_left_camera_frame, origin xyz=0 0.0315 0 rpy=0 0 0
- added joint zed_left_camera_optical_joint: type fixed, parent zed_left_camera_frame, child zed_left_camera_optical_frame, origin xyz=0 0 0 rpy=-1.57079632679 0.0 -1.57079632679
- added joint zed_right_camera_joint: type fixed, parent zed_camera_center, child zed_right_camera_frame, origin xyz=0 -0.0315 0 rpy=0 0 0
- added joint zed_right_camera_optical_joint: type fixed, parent zed_right_camera_frame, child zed_right_camera_optical_frame, origin xyz=0 0 0 rpy=-1.57079632679 0.0 -1.57079632679

File: ffw_description/urdf/ffw_sh5_rev1_follower/ffw_sh5_follower.urdf (robot description, URDF)
Before this commit: robot ffw_sh5_follower, 92 links, 91 joints
Links:
- removed link camera_l_bottom_screw_frame
- removed link camera_l_link
- removed link camera_r_bottom_screw_frame
- removed link camera_r_link
- removed link zedm_camera_center
- removed link zedm_camera_link
- removed link zedm_left_camera_frame
- removed link zedm_left_camera_optical_frame
- removed link zedm_right_camera_frame
- removed link zedm_right_camera_optical_frame
- added link camera_left_bottom_screw_frame
- added link camera_left_link, mass 0.072; collision box size=0.023 0.042 0.042; visual mesh filename=file:///root/ros2_ws/install/realsense2_description/share/r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 scale=0.001 0.001 0.001
- added link camera_right_bottom_screw_frame
- added link camera_right_link, mass 0.072; collision box size=0.023 0.042 0.042; visual mesh filename=file:///root/ros2_ws/install/realsense2_description/share/r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 scale=0.001 0.001 0.001
- added link zed_camera_center; collision mesh filename=package://ffw_description/meshes/common/follower/zedm.stl scale=0.001 0.001 0.001; visual mesh filename=package://ffw_description/meshes/common/follower/zedm.stl scale=0.001 0.001 0.001
- added link zed_camera_link
- added link zed_left_camera_frame
- added link zed_left_camera_optical_frame
- added link zed_right_camera_frame
- added link zed_right_camera_optical_frame
Joints:
- removed joint camera_l_joint
- removed joint camera_l_link_joint
- removed joint camera_r_joint
- removed joint camera_r_link_joint
- removed joint zedm_camera_center_joint
- removed joint zedm_joint
- removed joint zedm_left_camera_joint
- removed joint zedm_left_camera_optical_joint
- removed joint zedm_right_camera_joint
- removed joint zedm_right_camera_optical_joint
- added joint camera_left_joint: type fixed, parent arm_l_link7, child camera_left_bottom_screw_frame, origin xyz=0.108236 -0.021 -0.062552 rpy=-1.57079632679 1.66678943569 0
- added joint camera_left_link_joint: type fixed, parent camera_left_bottom_screw_frame, child camera_left_link, origin xyz=0.01085 0.009 0.021 rpy=0 0 0
- added joint camera_right_joint: type fixed, parent arm_r_link7, child camera_right_bottom_screw_frame, origin xyz=0.108236 -0.021 -0.062552 rpy=-1.57079632679 1.66678943569 0
- added joint camera_right_link_joint: type fixed, parent camera_right_bottom_screw_frame, child camera_right_link, origin xyz=0.01085 0.009 0.021 rpy=0 0 0
- added joint zed_camera_center_joint: type fixed, parent zed_camera_link, child zed_camera_center, origin xyz=0 0 0.01325 rpy=0 0 0
- added joint zed_joint: type fixed, parent head_link2, child zed_camera_link, origin xyz=0.0238122 -0.00651797 -0.0242094 rpy=0 0 0
- added joint zed_left_camera_joint: type fixed, parent zed_camera_center, child zed_left_camera_frame, origin xyz=0 0.0315 0 rpy=0 0 0
- added joint zed_left_camera_optical_joint: type fixed, parent zed_left_camera_frame, child zed_left_camera_optical_frame, origin xyz=0 0 0 rpy=-1.57079632679 0.0 -1.57079632679
- added joint zed_right_camera_joint: type fixed, parent zed_camera_center, child zed_right_camera_frame, origin xyz=0 -0.0315 0 rpy=0 0 0
- added joint zed_right_camera_optical_joint: type fixed, parent zed_right_camera_frame, child zed_right_camera_optical_frame, origin xyz=0 0 0 rpy=-1.57079632679 0.0 -1.57079632679
