Commit message: Added inertial and visual for sh5 lidar links

File: ffw_description/urdf/ffw_sh5_rev1_follower/ffw_sh5_follower.urdf.xacro (robot description, xacro)
@@ -48,4 +48,13 @@
   </joint>
   <link name="$(arg prefix)lidar_l_link">
+    <inertial>
+      <mass value="0.1"/>
+      <inertia ixx="0.0001" ixy="0" ixz="0" iyy="0.0001" iyz="0" izz="0.0001"/>
+    </inertial>
+    <visual>
+      <geometry>
+        <cylinder radius="0.03" length="0.03"/>
+      </geometry>
+    </visual>
   </link>
   <joint name="$(arg prefix)lidar_r_joint" type="fixed">
@@ -55,4 +64,15 @@
   </joint>
   <link name="$(arg prefix)lidar_r_link">
+    <inertial>
+      <mass value="0.1"/>
+      <origin xyz="0 0 0" rpy="0 0 0"/>
+      <inertia ixx="0.0001" ixy="0" ixz="0" iyy="0.0001" iyz="0" izz="0.0001"/>
+    </inertial>
+    <visual>
+      <geometry>
+        <cylinder radius="0.03" length="0.03"/>
+      </geometry>
+      <material name="blue"><color rgba="0 0 1 1"/></material>
+    </visual>
   </link>
   <joint name="$(arg prefix)imu_joint" type="fixed">
