Commit message: Update URDFS

File: ffw_description/urdf/ffw_sh5_rev1_follower/ffw_sh5_follower.urdf (robot description, URDF)
Before this commit: robot ffw_sh5_follower, 90 links, 89 joints
Links:
- added link end_effector_l_link; visual box size=0.01 0.01 0.01
- added link end_effector_r_link; visual box size=0.01 0.01 0.01
- link arm_base_link: geometry collision mesh filename=package://ffw_description/meshes/common/follower/ffw/body_a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 scale=0.001 0.001 0.001; visual mesh filename=package://ffw_description/meshes/common/follower/ffw/body_a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 scale=0.001 0.001 0.001
- link arm_l_link1: geometry collision mesh filename=package://ffw_description/meshes/common/follower/ffw/arm_l_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 scale=0.001 0.001 0.001; visual mesh filename=package://ffw_description/meshes/common/follower/ffw/arm_l_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 scale=0.001 0.001 0.001
- link arm_l_link2: geometry collision mesh filename=package://ffw_description/meshes/common/follower/ffw/arm_l_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 scale=0.001 0.001 0.001; visual mesh filename=package://ffw_description/meshes/common/follower/ffw/arm_l_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 scale=0.001 0.001 0.001
- link arm_l_link3: geometry collision mesh filename=package://ffw_description/meshes/common/follower/ffw/arm_l_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 scale=0.001 0.001 0.001; visual mesh filename=package://ffw_description/meshes/common/follower/ffw/arm_l_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 scale=0.001 0.001 0.001
- link arm_l_link4: geometry collision mesh filename=package://ffw_description/meshes/common/follower/ffw/arm_l_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 scale=0.001 0.001 0.001; visual mesh filename=package://ffw_description/meshes/common/follower/ffw/arm_l_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 scale=0.001 0.001 0.001
- link arm_l_link5: geometry collision mesh filename=package://ffw_description/meshes/common/follower/ffw/arm_l_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 scale=0.001 0.001 0.001; visual mesh filename=package://ffw_description/meshes/common/follower/ffw/arm_l_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 scale=0.001 0.001 0.001
- link arm_l_link6: geometry collision mesh filename=package://ffw_description/meshes/common/follower/ffw/arm_l_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 scale=0.001 0.001 0.001; visual mesh filename=package://ffw_description/meshes/common/follower/ffw/arm_l_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 scale=0.001 0.001 0.001
- link arm_l_link7: geometry collision mesh filename=package://ffw_description/meshes/common/follower/ffw/arm_l_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 scale=0.001 0.001 0.001; visual mesh filename=package://ffw_description/meshes/common/follower/ffw/arm_l_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 scale=0.001 0.001 0.001
- link arm_r_link1: geometry collision mesh filename=package://ffw_description/meshes/common/follower/ffw/arm_r_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 scale=0.001 0.001 0.001; visual mesh filename=package://ffw_description/meshes/common/follower/ffw/arm_r_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 scale=0.001 0.001 0.001
- link arm_r_link2: geometry collision mesh filename=package://ffw_description/meshes/common/follower/ffw/arm_r_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 scale=0.001 0.001 0.001; visual mesh filename=package://ffw_description/meshes/common/follower/ffw/arm_r_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 scale=0.001 0.001 0.001
- link arm_r_link3: geometry collision mesh filename=package://ffw_description/meshes/common/follower/ffw/arm_r_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 scale=0.001 0.001 0.001; visual mesh filename=package://ffw_description/meshes/common/follower/ffw/arm_r_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 scale=0.001 0.001 0.001
- link arm_r_link4: geometry collision mesh filename=package://ffw_description/meshes/common/follower/ffw/arm_r_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 scale=0.001 0.001 0.001; visual mesh filename=package://ffw_description/meshes/common/follower/ffw/arm_r_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 scale=0.001 0.001 0.001
- link arm_r_link5: geometry collision mesh filename=package://ffw_description/meshes/common/follower/ffw/arm_r_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 scale=0.001 0.001 0.001; visual mesh filename=package://ffw_description/meshes/common/follower/ffw/arm_r_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 scale=0.001 0.001 0.001
- link arm_r_link6: geometry collision mesh filename=package://ffw_description/meshes/common/follower/ffw/arm_r_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 scale=0.001 0.001 0.001; visual mesh filename=package://ffw_description/meshes/common/follower/ffw/arm_r_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 scale=0.001 0.001 0.001
- link arm_r_link7: geometry collision mesh filename=package://ffw_description/meshes/common/follower/ffw/arm_r_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 scale=0.001 0.001 0.001; visual mesh filename=package://ffw_description/meshes/common/follower/ffw/arm_r_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 scale=0.001 0.001 0.001
- link base_link: mass 35.989 -> 3.598943900e+01; geometry collision mesh filename=package://ffw_description/meshes/common/follower/ffw_swerve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 scale=0.001 0.001 0.001; visual mesh filename=package://ffw_description/meshes/common/follower/ffw_swerve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 scale=0.001 0.001 0.001
- link head_link1: geometry collision mesh filename=package://ffw_description/meshes/common/follower/ffw/head_l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 scale=0.001 0.001 0.001; visual mesh filename=package://ffw_description/meshes/common/follower/ffw/head_l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 scale=0.001 0.001 0.001
- link head_link2: geometry collision mesh filename=package://ffw_description/meshes/common/follower/ffw/head_l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 scale=0.001 0.001 0.001; visual mesh filename=package://ffw_description/meshes/common/follower/ffw/head_l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 scale=0.001 0.001 0.001
- link left_wheel_drive_link: geometry collision cylinder length=0.05 radius=0.0865; visual mesh filename=package://ffw_description/meshes/common/follower/ffw_swerve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 scale=0.001 0.001 0.001
- link left_wheel_steer_link: geometry collision mesh filename=package://ffw_description/meshes/common/follower/ffw_swerve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 scale=0.001 0.001 0.001; visual mesh filename=package://ffw_description/meshes/common/follower/ffw_swerve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 scale=0.001 0.001 0.001
- link lift_link: mass 1.790000000e+01 -> 17.9; geometry collision mesh filename=package://ffw_description/meshes/common/follower/ffw_swerve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 scale=0.001 0.001 0.001; visual mesh filename=package://ffw_description/meshes/common/follower/ffw_swerve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 scale=0.001 0.001 0.001
- link rear_wheel_drive_link: geometry collision cylinder length=0.05 radius=0.0865; visual mesh filename=package://ffw_description/meshes/common/follower/ffw_swerve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 scale=0.001 0.001 0.001
- link rear_wheel_steer_link: geometry collision mesh filename=package://ffw_description/meshes/common/follower/ffw_swerve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 scale=0.001 0.001 0.001; visual mesh filename=package://ffw_description/meshes/common/follower/ffw_swerve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 scale=0.001 0.001 0.001
- link right_wheel_drive_link: geometry collision cylinder length=0.05 radius=0.0865; visual mesh filename=package://ffw_description/meshes/common/follower/ffw_swerve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 scale=0.001 0.001 0.001
- link right_wheel_steer_link: geometry collision mesh filename=package://ffw_description/meshes/common/follower/ffw_swerve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 scale=0.001 0.001 0.001; visual mesh filename=package://ffw_description/meshes/common/follower/ffw_swerve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 scale=0.001 0.001 0.001
Joints:
- added joint l_palm: type fixed, parent hx5_d20_left_base, child end_effector_l_link, origin xyz=0.0 0.0 0.054 rpy=0 0 0
- added joint r_palm: type fixed, parent hx5_d20_right_base, child end_effector_r_link, origin xyz=0.0 0.0 0.054 rpy=0 0 0
