Commit message: Update leader parameters
Signed-off-by: cmk-robotis <cmk@robotis.com>

File: ffw_description/ros2_control/ffw_lg2_mini_leader/ffw_lg2_mini_leader_left.ros2_control.xacro (robot description, xacro)
@@ -74,5 +74,5 @@
       <gpio name="sensorxel_l_joy">
         <param name="type">sensor</param>
-        <param name="ID">10</param>
+        <param name="ID">40</param>
         <state_interface name="JOYSTICK X VALUE"/>
         <state_interface name="JOYSTICK Y VALUE"/>

File: ffw_description/ros2_control/ffw_lg2_mini_leader/ffw_lg2_mini_leader_left.ros2_control_orig.xacro (robot description, xacro)
@@ -74,5 +74,5 @@
       <gpio name="sensorxel_l_joy">
         <param name="type">sensor</param>
-        <param name="ID">10</param>
+        <param name="ID">40</param>
         <state_interface name="JOYSTICK X VALUE"/>
         <state_interface name="JOYSTICK Y VALUE"/>

File: ffw_description/urdf/ffw_lg2_mini_leader/ffw_lg2_mini_leader.urdf.xacro (robot description, xacro)
@@ -5,27 +5,11 @@
   <xacro:arg name="mock_sensor_commands" default="false" />
   <xacro:arg name="prefix" default="" />
-  <xacro:include filename="$(find ffw_description)/urdf/leader/ffw_leader_body.urdf.xacro" />
+  <xacro:include filename="$(find ffw_description)/urdf/leader/ffw_mini_leader_body.urdf.xacro" />
   <xacro:include filename="$(find ffw_description)/ros2_control/ffw_lg2_mini_leader/ffw_lg2_mini_leader_left.ros2_control.xacro" />
   <xacro:include filename="$(find ffw_description)/ros2_control/ffw_lg2_mini_leader/ffw_lg2_mini_leader_right.ros2_control.xacro" />
   <link name="world"/>
-  <xacro:ffw_leader_body parent="$(arg prefix)world" prefix="$(arg prefix)">
+  <xacro:ffw_mini_leader_body parent="$(arg prefix)world" prefix="$(arg prefix)">
     <origin xyz="0 0 0" rpy="0 0 0" />
-  </xacro:ffw_leader_body>
-  <joint name="$(arg prefix)gripper_l_joint1" type="revolute">
-    <origin xyz="0 0 0" rpy="0 0 0"/>
-    <parent link="$(arg prefix)arm_l_link7"/>
-    <axis xyz="0 1 0"/>
-    <child link="$(arg prefix)gripper_l_link1"/>
-    <limit velocity="6.5" effort="1000" lower="-6.28" upper="6.28" />
-  </joint>
-  <link name="$(arg prefix)gripper_l_link1"/>
-  <joint name="$(arg prefix)gripper_r_joint1" type="revolute">
-    <origin xyz="0 0 0" rpy="0 0 0"/>
-    <parent link="$(arg prefix)arm_r_link7"/>
-    <axis xyz="0 1 0"/>
-    <child link="$(arg prefix)gripper_r_link1"/>
-    <limit velocity="6.5" effort="1000" lower="-6.28" upper="6.28" />
-  </joint>
-  <link name="$(arg prefix)gripper_r_link1"/>
+  </xacro:ffw_mini_leader_body>
   <xacro:ffw_lg2_mini_leader_left_system
       use_sim="$(arg use_sim)"
