Commit message: Increase head joint limit
Signed-off-by: 20CMK <minkwon157@tukorea.ac.kr>

File: ffw_description/urdf/common/follower/ffw_follower_body.xacro (robot description, xacro)
@@ -42,5 +42,6 @@
          <origin xyz="0.049483 0 0.102130" rpy="0 0 0" />
          <axis xyz="0 1 0" />
-         <limit velocity="4.8" effort="1000" lower="-0.2317" upper="0.6951" />
+         <!-- <limit velocity="4.8" effort="1000" lower="-0.2317" upper="0.6951" /> -->
+         <limit velocity="4.8" effort="1000" lower="-0.2317" upper="0.83" />
          <dynamics damping="0.1" />
       </joint>
