Commit message: Replaced gripper with hx2-d1

File: ffw_description/urdf/common/follower/ffw_f_follower_body.xacro (robot description, xacro)
@@ -300,5 +300,5 @@
          <parent link="${prefix}arm_l_link6" />
          <child link="${prefix}arm_l_link7" />
-         <origin xyz="0 -0.0007 -0.0775" rpy="0 0 0" />
+         <origin xyz="-0.00025 -0.0007 -0.0775" rpy="0 0 0" />
          <axis xyz="1 0 0" />
          <limit velocity="4.8" effort="1000" lower="-1.8201" upper="1.5804" />
@@ -329,7 +329,7 @@
          </inertial>
       </link>
-      <xacro:sensor_d405 parent="${prefix}arm_l_link7" use_nominal_extrinsics="false" name="${prefix}camera_l">
+      <!-- <xacro:sensor_d405 parent="${prefix}arm_l_link7" use_nominal_extrinsics="false" name="${prefix}camera_l">
          <origin xyz="0.108236 -0.021 -0.062552" rpy="-1.57079632679 1.66678943569 0"/>
-      </xacro:sensor_d405>
+      </xacro:sensor_d405> -->
       <joint name="${prefix}arm_r_joint1" type="revolute">
          <parent link="${prefix}arm_base_link" />
@@ -556,7 +556,7 @@
          </inertial>
       </link>
-      <xacro:sensor_d405 parent="${prefix}arm_r_link7" use_nominal_extrinsics="false" name="${prefix}camera_r">
+      <!-- <xacro:sensor_d405 parent="${prefix}arm_r_link7" use_nominal_extrinsics="false" name="${prefix}camera_r">
          <origin xyz="0.108236 -0.021 -0.062552" rpy="-1.57079632679 1.66678943569 0"/>
-      </xacro:sensor_d405>
+      </xacro:sensor_d405> -->
    </xacro:macro>
 </robot>

File: ffw_description/urdf/ffw_f1_follower/ffw_f1_follower.urdf.xacro (robot description, xacro)
@@ -10,6 +10,5 @@
   <xacro:arg name="ros2_control_type" default="ffw_f1_follower" />
   <xacro:include filename="$(find ffw_description)/urdf/common/follower/ffw_f_follower_body.xacro" />
-  <!-- TODO: Change gripper to hx2_d1 -->
-  <xacro:include filename="$(find ffw_description)/urdf/common/rh_p12_rn_a/rh_p12_rn_a.urdf.xacro" />
+  <xacro:include filename="$(find ffw_description)/urdf/common/hx2_d1/hx2_d1.urdf.xacro" />
   <xacro:include filename="$(find ffw_description)/ros2_control/$(arg model)/$(arg ros2_control_type).ros2_control.xacro" />
   <xacro:include filename="$(find ffw_description)/gazebo/$(arg model)/ffw_f1_follower.gazebo.xacro" />
@@ -47,12 +46,11 @@
     <origin xyz="0.0055 0 1.4316" rpy="0 0 0" />
   </xacro:ffw_f_follower_body>
-  <!-- TODO: Change gripper to hx2_d1 -->
-  <xacro:rh_p12_rn_a parent="$(arg prefix)arm_l_link7" prefix="$(arg prefix)gripper_l_">
-    <origin xyz="0 0 -0.078" rpy="0 3.14159265359 3.14159265359"/>
-  </xacro:rh_p12_rn_a>
+  <xacro:hx2_d1 parent="$(arg prefix)arm_l_link7" prefix="$(arg prefix)gripper_l_">
+    <origin xyz="0.00025 0 -0.049" rpy="0 3.14159265359 3.14159265359"/>
+  </xacro:hx2_d1>
   <joint name="$(arg prefix)end_effector_l_joint" type="fixed">
     <parent link="$(arg prefix)arm_l_link7"/>
     <child link="$(arg prefix)end_effector_l_link"/>
-    <origin xyz="0 0 -0.215" rpy="0 0 0"/>
+    <origin xyz="0 0 -0.186" rpy="0 0 0"/>
   </joint>
   <link name="$(arg prefix)end_effector_l_link">
@@ -67,12 +65,11 @@
     </visual>
   </link>
-  <!-- TODO: Change gripper to hx2_d1 -->
-  <xacro:rh_p12_rn_a parent="$(arg prefix)arm_r_link7" prefix="$(arg prefix)gripper_r_">
-    <origin xyz="0 0 -0.078" rpy="0 3.14159265359 3.14159265359"/>
-  </xacro:rh_p12_rn_a>
+  <xacro:hx2_d1 parent="$(arg prefix)arm_r_link7" prefix="$(arg prefix)gripper_r_">
+    <origin xyz="0.00025 0 -0.049" rpy="0 3.14159265359 3.14159265359"/>
+  </xacro:hx2_d1>
   <joint name="$(arg prefix)end_effector_r_joint" type="fixed">
     <parent link="$(arg prefix)arm_r_link7"/>
     <child link="$(arg prefix)end_effector_r_link"/>
-    <origin xyz="0 0 -0.215" rpy="0 0 0"/>
+    <origin xyz="0 0 -0.186" rpy="0 0 0"/>
   </joint>
   <link name="$(arg prefix)end_effector_r_link">

File: ffw_description/urdf/ffw_f2_follower/ffw_f2_follower.urdf.xacro (robot description, xacro)
@@ -10,6 +10,5 @@
   <xacro:arg name="ros2_control_type" default="ffw_f2_follower" />
   <xacro:include filename="$(find ffw_description)/urdf/common/follower/ffw_f_follower_body.xacro" />
-  <!-- TODO: Change gripper to hx2_d1 -->
-  <xacro:include filename="$(find ffw_description)/urdf/common/rh_p12_rn_a/rh_p12_rn_a.urdf.xacro" />
+  <xacro:include filename="$(find ffw_description)/urdf/common/hx2_d1/hx2_d1.urdf.xacro" />
   <xacro:include filename="$(find ffw_description)/ros2_control/$(arg model)/$(arg ros2_control_type).ros2_control.xacro" />
   <xacro:include filename="$(find ffw_description)/ros2_control/$(arg model)/ffw_f2_base.ros2_control.xacro" />
@@ -117,12 +116,11 @@
     <origin xyz="-0.0753807 0 1.407" rpy="0 0 0" />
   </xacro:ffw_f_follower_body>
-  <!-- TODO: Change gripper to hx2_d1 -->
-  <xacro:rh_p12_rn_a parent="$(arg prefix)arm_l_link7" prefix="$(arg prefix)gripper_l_">
-    <origin xyz="0 0 -0.078" rpy="0 3.14159265359 3.14159265359"/>
-  </xacro:rh_p12_rn_a>
+  <xacro:hx2_d1 parent="$(arg prefix)arm_l_link7" prefix="$(arg prefix)gripper_l_">
+    <origin xyz="0.00025 0 -0.049" rpy="0 3.14159265359 3.14159265359"/>
+  </xacro:hx2_d1>
   <joint name="$(arg prefix)end_effector_l_joint" type="fixed">
     <parent link="$(arg prefix)arm_l_link7"/>
     <child link="$(arg prefix)end_effector_l_link"/>
-    <origin xyz="0 0 -0.215" rpy="0 0 0"/>
+    <origin xyz="0 0 -0.186" rpy="0 0 0"/>
   </joint>
   <link name="$(arg prefix)end_effector_l_link">
@@ -137,12 +135,11 @@
     </visual>
   </link>
-  <!-- TODO: Change gripper to hx2_d1 -->
-  <xacro:rh_p12_rn_a parent="$(arg prefix)arm_r_link7" prefix="$(arg prefix)gripper_r_">
-    <origin xyz="0 0 -0.078" rpy="0 3.14159265359 3.14159265359"/>
-  </xacro:rh_p12_rn_a>
+  <xacro:hx2_d1 parent="$(arg prefix)arm_r_link7" prefix="$(arg prefix)gripper_r_">
+    <origin xyz="0.00025 0 -0.049" rpy="0 3.14159265359 3.14159265359"/>
+  </xacro:hx2_d1>
   <joint name="$(arg prefix)end_effector_r_joint" type="fixed">
     <parent link="$(arg prefix)arm_r_link7"/>
     <child link="$(arg prefix)end_effector_r_link"/>
-    <origin xyz="0 0 -0.215" rpy="0 0 0"/>
+    <origin xyz="0 0 -0.186" rpy="0 0 0"/>
   </joint>
   <link name="$(arg prefix)end_effector_r_link">

Commit message: Modified inertials

File: ffw_description/urdf/common/follower/ffw_f_follower_body.xacro (robot description, xacro)
@@ -322,9 +322,9 @@
          </collision>
          <inertial>
-            <origin xyz="2.550659300e-02 0.000000000e+00 -5.539533100e-02" />
-            <mass value="1.668563000e-01" />
-            <inertia ixx="1.035867900e-04" ixy="0.000000000e+00" ixz="1.098870100e-05"
-            iyy="4.524528700e-04" iyz="0.000000000e+00"
-            izz="4.156884400e-04" />
+            <origin xyz="5.0778477e-03  0.0000000e-03 -3.1576679e-02" />
+            <mass value="1.4594797e-01" />
+            <inertia ixx="7.6276195e-05" ixy="0.000000000e+00" ixz="6.4673549e-06"
+            iyy="2.4260619e-04" iyz="0.000000000e+00"
+            izz="2.2469260e-04" />
          </inertial>
       </link>
@@ -549,9 +549,9 @@
          </collision>
          <inertial>
-            <origin xyz="2.546836200e-02 1.396001200e-03 -5.539533100e-02" />
-            <mass value="1.668563000e-01" />
-            <inertia ixx="1.046318100e-04" ixy="-1.906515900e-05" ixz="1.097223300e-05"
-            iyy="4.514078500e-04" iyz="6.013716400e-07"
-            izz="4.156884400e-04" />
+            <origin xyz="5.0778477e-03  0.0000000e-03 -3.1576679e-02" />
+            <mass value="1.4594797e-01" />
+            <inertia ixx="7.6276195e-05" ixy="0.000000000e+00" ixz="6.4673549e-06"
+            iyy="2.4260619e-04" iyz="0.000000000e+00"
+            izz="2.2469260e-04" />
          </inertial>
       </link>

File: ffw_description/urdf/common/hx2_d1/hx2_d1.urdf.xacro (robot description, xacro)
@@ -29,7 +29,7 @@
       </visual>
       <inertial>
-        <origin xyz="0.000 0.000 0.032" rpy="0 0 0"/>
-        <mass value="0.236"/>
-        <inertia ixx="0.000001" ixy="0.0" ixz="0.0" iyy="0.000001" iyz="0.0" izz="0.000001" />
+        <origin xyz="-6.8484893e-05  0.0000000e+00  3.0231995e-02" rpy="0 0 0"/>
+        <mass value="2.1967564e-01"/>
+        <inertia ixx="1.4908617e-04" ixy="0.0" ixz="8.0082096e-07" iyy="1.1107191e-04" iyz="0.0" izz="1.5613575e-04" />
       </inertial>
     </link>
@@ -61,7 +61,7 @@
       </visual>
       <inertial>
-        <origin xyz="0.000 0.034 0.004" rpy="0 0 0"/>
-        <mass value="0.068"/>
-        <inertia ixx="0.000001" ixy="0.0" ixz="0.0" iyy="0.000001" iyz="0.0" izz="0.000001" />
+        <origin xyz="0.0000000e+00  3.3664697e-02  3.3231280e-03" rpy="0 0 0"/>
+        <mass value="2.1057910e-02"/>
+        <inertia ixx="1.1229445e-05" ixy="0.0" ixz="0.0" iyy="6.6539794e-06" iyz="-1.9651419e-06" izz="7.6921770e-06" />
       </inertial>
     </link>
@@ -70,5 +70,5 @@
       <parent link="${prefix}hx2_d1_r1"/>
       <child link="${prefix}hx2_d1_r2"/>
-      <origin xyz="0.0 0.0601042 0.0176601" rpy="0 0 0"/>
+      <origin xyz="0.0 0.0494977 0.0282667" rpy="0 0 0"/>
       <axis xyz="-1 0 0"/>
       <limit velocity="6.5" effort="1000" lower="0.0" upper="1.0" />
@@ -94,7 +94,7 @@
       </visual>
       <inertial>
-        <origin xyz="0.000 0.006 0.011" rpy="0 0 0"/>
-        <mass value="0.022"/>
-        <inertia ixx="0.000001" ixy="0.0" ixz="0.0" iyy="0.000001" iyz="0.0" izz="0.000001" />
+        <origin xyz="0.0000000e+00 -3.5851422e-03  2.3385920e-02" rpy="0 0 0"/>
+        <mass value="8.7352051e-02"/>
+        <inertia ixx="1.9038449e-05" ixy="0.0" ixz="0.0" iyy="2.1456514e-05" iyz="4.1006291e-06" izz="7.4235992e-06" />
       </inertial>
     </link>
@@ -127,7 +127,7 @@
       </visual>
       <inertial>
-        <origin xyz="0.000 -0.034 0.004" rpy="0 0 0"/>
-        <mass value="0.068"/>
-        <inertia ixx="0.000001" ixy="0.0" ixz="0.0" iyy="0.000001" iyz="0.0" izz="0.000001" />
+        <origin xyz="0.0000000e+00 -3.1948616e-02  1.8581523e-03" rpy="0 0 0"/>
+        <mass value="1.8933866e-02"/>
+        <inertia ixx="1.0233707e-05" ixy="0.0" ixz="0.0" iyy="6.0862054e-06" iyz="1.4864276e-06" izz="6.9498404e-06" />
       </inertial>
     </link>
@@ -136,5 +136,5 @@
       <parent link="${prefix}hx2_d1_l1"/>
       <child link="${prefix}hx2_d1_l2"/>
-      <origin xyz="0.0 -0.0601042 0.0176601" rpy="0 0 0"/>
+      <origin xyz="0.0 -0.0494977 0.0282667" rpy="0 0 0"/>
       <axis xyz="1 0 0"/>
       <limit velocity="6.5" effort="1000" lower="0.0" upper="1.0" />
@@ -160,7 +160,7 @@
       </visual>
       <inertial>
-        <origin xyz="0.000 -0.006 0.011" rpy="0 0 0"/>
-        <mass value="0.022"/>
-        <inertia ixx="0.000001" ixy="0.0" ixz="0.0" iyy="0.000001" iyz="0.0" izz="0.000001" />
+        <origin xyz="0.0000000e+00 -6.7070088e-03  1.1261741e-02" rpy="0 0 0"/>
+        <mass value="9.5399014e-02"/>
+        <inertia ixx="2.1847544e-05" ixy="0.0" ixz="0.0" iyy="2.4457514e-05" iyz="-3.7396106e-06" izz="8.1383191e-06" />
       </inertial>
     </link>

Commit message: Added wrist camera

File: ffw_description/urdf/common/follower/ffw_f_follower_body.xacro (robot description, xacro)
@@ -2,5 +2,5 @@
 <robot xmlns:xacro="http://www.ros.org/wiki/xacro">
    <xacro:macro name="ffw_f_follower_body" params="prefix parent *origin">
-      <xacro:include filename="$(find realsense2_description)/urdf/_d405.urdf.xacro" />
+      <xacro:include filename="$(find ffw_description)/urdf/common/follower/wrist_d401.urdf.xacro" />
       <xacro:include filename="$(find realsense2_description)/urdf/_d455.urdf.xacro" />
       <xacro:property name="meshes_file_direction" value="package://ffw_description/meshes/common/follower/ffw_f" />
@@ -101,5 +101,4 @@
          </inertial>
       </link>
-      <!-- TODO : Modify camera name -->
       <xacro:sensor_d455 parent="${prefix}head_link2" use_nominal_extrinsics="false" name="${prefix}camera_head">
          <origin xyz="0.032705 0 -0.0025" rpy="0 0 0"/>
@@ -329,7 +328,7 @@
          </inertial>
       </link>
-      <!-- <xacro:sensor_d405 parent="${prefix}arm_l_link7" use_nominal_extrinsics="false" name="${prefix}camera_l">
-         <origin xyz="0.108236 -0.021 -0.062552" rpy="-1.57079632679 1.66678943569 0"/>
-      </xacro:sensor_d405> -->
+      <xacro:wrist_d401 parent="${prefix}arm_l_link7" name="${prefix}camera_l">
+         <origin xyz="0.0275 0.0 -0.0847501" rpy="-1.57079632679 1.57079632679 0"/>
+      </xacro:wrist_d401>
       <joint name="${prefix}arm_r_joint1" type="revolute">
          <parent link="${prefix}arm_base_link" />
@@ -556,7 +555,7 @@
          </inertial>
       </link>
-      <!-- <xacro:sensor_d405 parent="${prefix}arm_r_link7" use_nominal_extrinsics="false" name="${prefix}camera_r">
-         <origin xyz="0.108236 -0.021 -0.062552" rpy="-1.57079632679 1.66678943569 0"/>
-      </xacro:sensor_d405> -->
+      <xacro:wrist_d401 parent="${prefix}arm_r_link7" name="${prefix}camera_r">
+         <origin xyz="0.0275 0.0 -0.0847501" rpy="-1.57079632679 1.57079632679 0"/>
+      </xacro:wrist_d401>
    </xacro:macro>
 </robot>
