Commit message: refactor(ffw_description/meshes): organize follower meshes by component
Signed-off-by: cmk-robotis <cmk@robotis.com>

File: ffw_description/urdf/common/follower/ffw_f_follower_body.xacro (robot description, xacro)
@@ -4,5 +4,5 @@
       <xacro:include filename="$(find ffw_description)/urdf/common/follower/wrist_d401.urdf.xacro" />
       <xacro:include filename="$(find realsense2_description)/urdf/_d455.urdf.xacro" />
-      <xacro:property name="meshes_file_direction" value="package://ffw_description/meshes/common/follower/ffw_f" />
+      <xacro:property name="meshes_file_direction" value="package://ffw_description/meshes/follower/body/ffw_f" />
       <joint name="${prefix}lift_joint" type="prismatic">
          <parent link="${parent}"/>

File: ffw_description/urdf/common/follower/ffw_follower_body.xacro (robot description, xacro)
@@ -4,5 +4,5 @@
       <xacro:include filename="$(find realsense2_description)/urdf/_d405.urdf.xacro" />
       <xacro:include filename="$(find ffw_description)/urdf/common/follower/zedm.urdf.xacro" />
-      <xacro:property name="meshes_file_direction" value="package://ffw_description/meshes/common/follower/ffw" />
+      <xacro:property name="meshes_file_direction" value="package://ffw_description/meshes/follower/body/ffw" />
       <joint name="${prefix}lift_joint" type="prismatic">
          <parent link="${parent}"/>

File: ffw_description/urdf/common/follower/wrist_d401.urdf.xacro (robot description, xacro)
@@ -10,5 +10,5 @@
 			<visual>
 				<geometry>
-					<mesh filename="file://$(find ffw_description)/meshes/common/follower/wrist_d401_base.stl" scale="0.001 0.001 0.001"/>
+					<mesh filename="file://$(find ffw_description)/meshes/follower/body/wrist_d401_base.stl" scale="0.001 0.001 0.001"/>
 				</geometry>
 				<material name="d401_black">
@@ -19,5 +19,5 @@
 				<origin xyz="0 0 0" rpy="0 0 0"/>
 				<geometry>
-					<mesh filename="file://$(find ffw_description)/meshes/common/follower/wrist_d401_base.stl" scale="0.001 0.001 0.001"/>
+					<mesh filename="file://$(find ffw_description)/meshes/follower/body/wrist_d401_base.stl" scale="0.001 0.001 0.001"/>
 				</geometry>
 			</collision>

File: ffw_description/urdf/common/follower/zedm.urdf.xacro (robot description, xacro)
@@ -7,5 +7,5 @@
 				<origin xyz="0 0 0" rpy="0 0 0"/>
 				<geometry>
-					<mesh filename="file://$(find ffw_description)/meshes/common/follower/zedm.stl" scale="0.001 0.001 0.001"/>
+					<mesh filename="file://$(find ffw_description)/meshes/follower/body/zedm.stl" scale="0.001 0.001 0.001"/>
 				</geometry>
 				<material name="zedm_mat">
@@ -16,5 +16,5 @@
 				<origin xyz="0 0 0" rpy="0 0 0"/>
 				<geometry>
-					<mesh filename="file://$(find ffw_description)/meshes/common/follower/zedm.stl" scale="0.001 0.001 0.001"/>
+					<mesh filename="file://$(find ffw_description)/meshes/follower/body/zedm.stl" scale="0.001 0.001 0.001"/>
 				</geometry>
 			</collision>

File: ffw_description/urdf/common/hx2_d1/hx2_d1.urdf.xacro (robot description, xacro)
@@ -5,5 +5,5 @@
     <xacro:property
       name="meshes_file_direction"
-      value="package://ffw_description/meshes/common/hx2_d1"/>
+      value="package://ffw_description/meshes/follower/gripper/hx2_d1"/>
     <joint name="${prefix}joint" type="fixed">
       <xacro:insert_block name="origin" />

File: ffw_description/urdf/common/hx5_d20/hx5_d20_left.urdf.xacro (robot description, xacro)
@@ -2,5 +2,5 @@
 <robot xmlns:xacro="http://www.ros.org/wiki/xacro">
    <xacro:macro name="hx5_d20_left" params="prefix parent *origin">
-      <xacro:property name="meshes_file_direction" value="package://ffw_description/meshes/common/hx5_d20/hx5_d20_left/" />
+      <xacro:property name="meshes_file_direction" value="package://ffw_description/meshes/follower/gripper/hx5_d20/hx5_d20_left/" />
       <joint name="${prefix}hx5_d20_left_joint" type="fixed">
          <xacro:insert_block name="origin" />

File: ffw_description/urdf/common/hx5_d20/hx5_d20_right.urdf.xacro (robot description, xacro)
@@ -2,5 +2,5 @@
 <robot xmlns:xacro="http://www.ros.org/wiki/xacro">
    <xacro:macro name="hx5_d20_right" params="prefix parent *origin">
-      <xacro:property name="meshes_file_direction" value="package://ffw_description/meshes/common/hx5_d20/hx5_d20_right/" />
+      <xacro:property name="meshes_file_direction" value="package://ffw_description/meshes/follower/gripper/hx5_d20/hx5_d20_right/" />
       <joint name="${prefix}hx5_d20_right_joint" type="fixed">
          <xacro:insert_block name="origin" />

File: ffw_description/urdf/common/rh_p12_rn_a/rh_p12_rn_a.urdf.xacro (robot description, xacro)
@@ -5,5 +5,5 @@
     <xacro:property
       name="meshes_file_direction"
-      value="package://ffw_description/meshes/common/rh_p12_rn_a"/>
+      value="package://ffw_description/meshes/follower/gripper/rh_p12_rn_a"/>
     <joint name="${prefix}joint" type="fixed">
       <xacro:insert_block name="origin" />

File: ffw_description/urdf/ffw_bg2_rev4_follower/ffw_bg2_follower.urdf.xacro (robot description, xacro)
@@ -1,6 +1,5 @@
 <?xml version="1.0"?>
 <robot xmlns:xacro="http://www.ros.org/wiki/xacro" name="ffw_bg2_follower">
-  <xacro:property name="meshes_file_direction" value="package://ffw_description/meshes/$(arg model)" />
-  <xacro:property name="base_meshes_dir" value="package://ffw_description/meshes/common/follower/ffw_base" />
+  <xacro:property name="base_meshes_dir" value="package://ffw_description/meshes/follower/base/ffw_base" />
   <xacro:arg name="use_sim" default="false" />
   <xacro:arg name="use_mock_hardware" default="false" />

File: ffw_description/urdf/ffw_bh5_rev1_follower/ffw_bh5_follower.urdf.xacro (robot description, xacro)
@@ -1,6 +1,5 @@
 <?xml version="1.0"?>
 <robot xmlns:xacro="http://www.ros.org/wiki/xacro" name="ffw_bh5_follower">
-  <xacro:property name="meshes_file_direction" value="package://ffw_description/meshes/$(arg model)" />
-  <xacro:property name="base_meshes_dir" value="package://ffw_description/meshes/common/follower/ffw_base" />
+  <xacro:property name="base_meshes_dir" value="package://ffw_description/meshes/follower/base/ffw_base" />
   <xacro:arg name="use_sim" default="false" />
   <xacro:arg name="use_mock_hardware" default="false" />

File: ffw_description/urdf/ffw_f1_follower/ffw_f1_follower.urdf.xacro (robot description, xacro)
@@ -1,6 +1,5 @@
 <?xml version="1.0"?>
 <robot xmlns:xacro="http://www.ros.org/wiki/xacro" name="ffw_f1_follower">
-  <xacro:property name="meshes_file_direction" value="package://ffw_description/meshes/$(arg model)" />
-  <xacro:property name="base_meshes_dir" value="package://ffw_description/meshes/common/follower/ffw_f_base" />
+  <xacro:property name="base_meshes_dir" value="package://ffw_description/meshes/follower/base/ffw_f_base" />
   <xacro:arg name="use_sim" default="false" />
   <xacro:arg name="use_mock_hardware" default="false" />

File: ffw_description/urdf/ffw_f2_follower/ffw_f2_follower.urdf.xacro (robot description, xacro)
@@ -1,6 +1,5 @@
 <?xml version="1.0"?>
 <robot xmlns:xacro="http://www.ros.org/wiki/xacro" name="ffw_f2_follower">
-  <xacro:property name="meshes_file_direction" value="package://ffw_description/meshes/$(arg model)" />
-  <xacro:property name="swerve_meshes_dir" value="package://ffw_description/meshes/common/follower/ffw_f_swerve" />
+  <xacro:property name="swerve_meshes_dir" value="package://ffw_description/meshes/follower/base/ffw_f_swerve" />
   <xacro:arg name="use_sim" default="false" />
   <xacro:arg name="use_mock_hardware" default="false" />

File: ffw_description/urdf/ffw_mobile_base/ffw_mobile_base.urdf.xacro (robot description, xacro)
@@ -1,6 +1,5 @@
 <?xml version="1.0"?>
 <robot xmlns:xacro="http://www.ros.org/wiki/xacro" name="ffw_mobile_base">
-  <xacro:property name="meshes_file_direction" value="package://ffw_description/meshes/$(arg model)" />
-  <xacro:property name="swerve_meshes_dir" value="package://ffw_description/meshes/common/follower/swerve" />
+  <xacro:property name="swerve_meshes_dir" value="package://ffw_description/meshes/follower/base/ffw_swerve" />
   <xacro:arg name="use_sim" default="false" />
   <xacro:arg name="use_mock_hardware" default="false" />

File: ffw_description/urdf/ffw_sg2_rev1_follower/ffw_sg2_follower.urdf.xacro (robot description, xacro)
@@ -1,6 +1,5 @@
 <?xml version="1.0"?>
 <robot xmlns:xacro="http://www.ros.org/wiki/xacro" name="ffw_sg2_follower">
-  <xacro:property name="meshes_file_direction" value="package://ffw_description/meshes/$(arg model)" />
-  <xacro:property name="swerve_meshes_dir" value="package://ffw_description/meshes/common/follower/ffw_swerve" />
+  <xacro:property name="swerve_meshes_dir" value="package://ffw_description/meshes/follower/base/ffw_swerve" />
   <xacro:arg name="use_sim" default="false" />
   <xacro:arg name="use_mock_hardware" default="false" />

File: ffw_description/urdf/ffw_sh5_rev1_follower/ffw_sh5_follower.urdf.xacro (robot description, xacro)
@@ -1,6 +1,5 @@
 <?xml version="1.0"?>
 <robot xmlns:xacro="http://www.ros.org/wiki/xacro" name="ffw_sh5_follower">
-  <xacro:property name="meshes_file_direction" value="package://ffw_description/meshes/$(arg model)" />
-  <xacro:property name="swerve_meshes_dir" value="package://ffw_description/meshes/common/follower/ffw_swerve" />
+  <xacro:property name="swerve_meshes_dir" value="package://ffw_description/meshes/follower/base/ffw_swerve" />
   <xacro:arg name="use_sim" default="false" />
   <xacro:arg name="use_mock_hardware" default="false" />
