Commit message: Modified xacros

File: ffw_description/urdf/common/follower/wrist_d401.urdf.xacro (robot description, xacro)
@@ -31,5 +31,5 @@
 			<parent link="${name}_base_link"/>
 			<child link="${name}_link"/>
-			<origin xyz="0.0126724 -0.02235 0.009" rpy="0 0 0" />
+			<origin xyz="0.0126724 -0.02235 0.009" rpy="0 0 0.3490656" />
 		</joint>
 		<link name="${name}_link" />

File: ffw_description/urdf/common/hx2_d1/hx2_d1.urdf.xacro (robot description, xacro)
@@ -94,7 +94,7 @@
       </visual>
       <inertial>
-        <origin xyz="0.0000000e+00 -3.5851422e-03  2.3385920e-02" rpy="0 0 0"/>
-        <mass value="8.7352051e-02"/>
-        <inertia ixx="1.9038449e-05" ixy="0.0" ixz="0.0" iyy="2.1456514e-05" iyz="4.1006291e-06" izz="7.4235992e-06" />
+        <origin xyz="0.0000000e+00 6.7070088e-03  1.1261741e-02" rpy="0 0 0"/>
+        <mass value="9.5399014e-02"/>
+        <inertia ixx="2.1847544e-05" ixy="0.0" ixz="0.0" iyy="2.4457514e-05" iyz="3.7396106e-06" izz="8.1383191e-06" />
       </inertial>
     </link>
