Commit message: Added prefix to world link

File: ffw_description/urdf/ffw_a2_leader/ffw_a2_leader.urdf.xacro (robot description, xacro)
@@ -7,5 +7,5 @@
   <xacro:include filename="$(find ffw_description)/urdf/common/leader/ffw_mini_leader_body.urdf.xacro" />
   <xacro:include filename="$(find ffw_description)/ros2_control/ffw_a2_leader/ffw_a2_leader.ros2_control.xacro" />
-  <link name="world"/>
+  <link name="$(arg prefix)world"/>
   <xacro:ffw_mini_leader_body parent="$(arg prefix)world" prefix="$(arg prefix)">
     <origin xyz="0 0 0" rpy="0 0 0" />
