Commit message: Fixed joint7 position limits

File: ffw_description/ros2_control/ffw_bg2_rev2_follower/ffw_bg2_follower.ros2_control.xacro (robot description, xacro)
@@ -348,6 +348,6 @@
         <param name="Profile Velocity">100</param>
         <param name="Profile Acceleration">50</param>
-        <param name="Max Position Limit">131875</param>
-        <param name="Min Position Limit">-131875</param>
+        <param name="Max Position Limit">152804</param>
+        <param name="Min Position Limit">-175979</param>
       </gpio>
       <gpio name="dxl8">
@@ -525,6 +525,6 @@
         <param name="Profile Velocity">100</param>
         <param name="Profile Acceleration">50</param>
-        <param name="Max Position Limit">131875</param>
-        <param name="Min Position Limit">-131875</param>
+        <param name="Max Position Limit">175979</param>
+        <param name="Min Position Limit">-152804</param>
       </gpio>
       <gpio name="dxl38">

File: ffw_description/ros2_control/ffw_bg2_rev3_follower/ffw_bg2_follower.ros2_control.xacro (robot description, xacro)
@@ -291,6 +291,6 @@
         <param name="Profile Velocity">2020</param>
         <param name="Profile Acceleration">3000</param>
-        <param name="Max Position Limit">151875</param>
-        <param name="Min Position Limit">-20000</param>
+        <param name="Max Position Limit">152804</param>
+        <param name="Min Position Limit">-175979</param>
       </gpio>
       <gpio name="dxl8">
@@ -428,6 +428,6 @@
         <param name="Profile Velocity">2020</param>
         <param name="Profile Acceleration">3000</param>
-        <param name="Max Position Limit">20000</param>
-        <param name="Min Position Limit">-151875</param>
+        <param name="Max Position Limit">175979</param>
+        <param name="Min Position Limit">-152804</param>
       </gpio>
       <gpio name="dxl38">

File: ffw_description/ros2_control/ffw_bg2_rev4_follower/ffw_bg2_follower.ros2_control.xacro (robot description, xacro)
@@ -306,6 +306,6 @@
         <param name="Profile Velocity">100</param>
         <param name="Profile Acceleration">50</param>
-        <param name="Max Position Limit">131875</param>
-        <param name="Min Position Limit">-151875</param>
+        <param name="Max Position Limit">152804</param>
+        <param name="Min Position Limit">-175979</param>
       </gpio>
       <gpio name="dxl8">
@@ -483,6 +483,6 @@
         <param name="Profile Velocity">100</param>
         <param name="Profile Acceleration">50</param>
-        <param name="Max Position Limit">131875</param>
-        <param name="Min Position Limit">-151875</param>
+        <param name="Max Position Limit">175979</param>
+        <param name="Min Position Limit">-152804</param>
       </gpio>
       <gpio name="dxl38">

File: ffw_description/ros2_control/ffw_bg2_rev4_follower/ffw_bg2_follower_smooth.ros2_control.xacro (robot description, xacro)
@@ -306,6 +306,6 @@
         <param name="Profile Velocity">300</param>
         <param name="Profile Acceleration">150</param>
-        <param name="Max Position Limit">131875</param>
-        <param name="Min Position Limit">-151875</param>
+        <param name="Max Position Limit">152804</param>
+        <param name="Min Position Limit">-175979</param>
       </gpio>
       <gpio name="dxl8">
@@ -483,6 +483,6 @@
         <param name="Profile Velocity">300</param>
         <param name="Profile Acceleration">150</param>
-        <param name="Max Position Limit">131875</param>
-        <param name="Min Position Limit">-151875</param>
+        <param name="Max Position Limit">175979</param>
+        <param name="Min Position Limit">-152804</param>
       </gpio>
       <gpio name="dxl38">

File: ffw_description/ros2_control/ffw_bh5_rev1_follower/ffw_bh5_follower.ros2_control.xacro (robot description, xacro)
@@ -1586,6 +1586,6 @@
         <param name="Profile Velocity">100</param>
         <param name="Profile Acceleration">50</param>
-        <param name="Max Position Limit">131875</param>
-        <param name="Min Position Limit">-151875</param>
+        <param name="Max Position Limit">152804</param>
+        <param name="Min Position Limit">-175979</param>
       </gpio>
       <!-- LEFT HAND -->
@@ -2652,6 +2652,6 @@
         <param name="Profile Velocity">100</param>
         <param name="Profile Acceleration">50</param>
-        <param name="Max Position Limit">131875</param>
-        <param name="Min Position Limit">-151875</param>
+        <param name="Max Position Limit">175979</param>
+        <param name="Min Position Limit">-152804</param>
       </gpio>
       <!-- LIFT -->

File: ffw_description/ros2_control/ffw_f1_follower/ffw_f1_follower.ros2_control.xacro (robot description, xacro)
@@ -306,6 +306,6 @@
         <param name="Profile Velocity">100</param>
         <param name="Profile Acceleration">50</param>
-        <param name="Max Position Limit">131875</param>
-        <param name="Min Position Limit">-151875</param>
+        <param name="Max Position Limit">152804</param>
+        <param name="Min Position Limit">-175979</param>
       </gpio>
       <gpio name="dxl8">
@@ -483,6 +483,6 @@
         <param name="Profile Velocity">100</param>
         <param name="Profile Acceleration">50</param>
-        <param name="Max Position Limit">131875</param>
-        <param name="Min Position Limit">-151875</param>
+        <param name="Max Position Limit">175979</param>
+        <param name="Min Position Limit">-152804</param>
       </gpio>
       <gpio name="dxl38">

File: ffw_description/ros2_control/ffw_f1_follower/ffw_f1_follower_smooth.ros2_control.xacro (robot description, xacro)
@@ -306,6 +306,6 @@
         <param name="Profile Velocity">300</param>
         <param name="Profile Acceleration">150</param>
-        <param name="Max Position Limit">131875</param>
-        <param name="Min Position Limit">-151875</param>
+        <param name="Max Position Limit">152804</param>
+        <param name="Min Position Limit">-175979</param>
       </gpio>
       <gpio name="dxl8">
@@ -483,6 +483,6 @@
         <param name="Profile Velocity">300</param>
         <param name="Profile Acceleration">150</param>
-        <param name="Max Position Limit">131875</param>
-        <param name="Min Position Limit">-151875</param>
+        <param name="Max Position Limit">175979</param>
+        <param name="Min Position Limit">-152804</param>
       </gpio>
       <gpio name="dxl38">

File: ffw_description/ros2_control/ffw_f2_follower/ffw_f2_follower.ros2_control.xacro (robot description, xacro)
@@ -325,6 +325,6 @@
         <param name="Profile Velocity">100</param>
         <param name="Profile Acceleration">50</param>
-        <param name="Max Position Limit">131875</param>
-        <param name="Min Position Limit">-151875</param>
+        <param name="Max Position Limit">152804</param>
+        <param name="Min Position Limit">-175979</param>
       </gpio>
       <gpio name="dxl8">
@@ -502,6 +502,6 @@
         <param name="Profile Velocity">100</param>
         <param name="Profile Acceleration">50</param>
-        <param name="Max Position Limit">131875</param>
-        <param name="Min Position Limit">-151875</param>
+        <param name="Max Position Limit">175979</param>
+        <param name="Min Position Limit">-152804</param>
       </gpio>
       <gpio name="dxl38">

File: ffw_description/ros2_control/ffw_f2_follower/ffw_f2_follower_smooth.ros2_control.xacro (robot description, xacro)
@@ -325,6 +325,6 @@
         <param name="Profile Velocity">300</param>
         <param name="Profile Acceleration">150</param>
-        <param name="Max Position Limit">131875</param>
-        <param name="Min Position Limit">-151875</param>
+        <param name="Max Position Limit">152804</param>
+        <param name="Min Position Limit">-175979</param>
       </gpio>
       <gpio name="dxl8">
@@ -502,6 +502,6 @@
         <param name="Profile Velocity">300</param>
         <param name="Profile Acceleration">150</param>
-        <param name="Max Position Limit">131875</param>
-        <param name="Min Position Limit">-151875</param>
+        <param name="Max Position Limit">175979</param>
+        <param name="Min Position Limit">-152804</param>
       </gpio>
       <gpio name="dxl38">

File: ffw_description/ros2_control/ffw_sg2_rev1_follower/ffw_sg2_follower.ros2_control.xacro (robot description, xacro)
@@ -325,6 +325,6 @@
         <param name="Profile Velocity">100</param>
         <param name="Profile Acceleration">50</param>
-        <param name="Max Position Limit">131875</param>
-        <param name="Min Position Limit">-151875</param>
+        <param name="Max Position Limit">152804</param>
+        <param name="Min Position Limit">-175979</param>
       </gpio>
       <gpio name="dxl8">
@@ -502,6 +502,6 @@
         <param name="Profile Velocity">100</param>
         <param name="Profile Acceleration">50</param>
-        <param name="Max Position Limit">131875</param>
-        <param name="Min Position Limit">-151875</param>
+        <param name="Max Position Limit">175979</param>
+        <param name="Min Position Limit">-152804</param>
       </gpio>
       <gpio name="dxl38">

File: ffw_description/ros2_control/ffw_sg2_rev1_follower/ffw_sg2_follower_smooth.ros2_control.xacro (robot description, xacro)
@@ -325,6 +325,6 @@
         <param name="Profile Velocity">300</param>
         <param name="Profile Acceleration">150</param>
-        <param name="Max Position Limit">131875</param>
-        <param name="Min Position Limit">-151875</param>
+        <param name="Max Position Limit">152804</param>
+        <param name="Min Position Limit">-175979</param>
       </gpio>
       <gpio name="dxl8">
@@ -502,6 +502,6 @@
         <param name="Profile Velocity">300</param>
         <param name="Profile Acceleration">150</param>
-        <param name="Max Position Limit">131875</param>
-        <param name="Min Position Limit">-151875</param>
+        <param name="Max Position Limit">175979</param>
+        <param name="Min Position Limit">-152804</param>
       </gpio>
       <gpio name="dxl38">

File: ffw_description/ros2_control/ffw_sh5_rev1_follower/ffw_sh5_follower.joints.xacro (robot description, xacro)
@@ -286,6 +286,6 @@
       <param name="Profile Velocity">100</param>
       <param name="Profile Acceleration">50</param>
-      <param name="Max Position Limit">131875</param>
-      <param name="Min Position Limit">-151875</param>
+      <param name="Max Position Limit">152804</param>
+      <param name="Min Position Limit">-175979</param>
     </gpio>
     <!-- LEFT ARM -->
@@ -450,6 +450,6 @@
       <param name="Profile Velocity">100</param>
       <param name="Profile Acceleration">50</param>
-      <param name="Max Position Limit">131875</param>
-      <param name="Min Position Limit">-151875</param>
+      <param name="Max Position Limit">175979</param>
+      <param name="Min Position Limit">-152804</param>
     </gpio>
     <!-- LIFT -->

File: ffw_description/urdf/common/follower/ffw_f_follower_body.xacro (robot description, xacro)
@@ -301,5 +301,5 @@
          <origin xyz="-0.00025 -0.0007 -0.0775" rpy="0 0 0" />
          <axis xyz="1 0 0" />
-         <limit velocity="4.8" effort="1000" lower="-1.8201" upper="1.5804" />
+         <limit velocity="4.8" effort="1000" lower="-1.5804" upper="1.8201" />
          <dynamics damping="0.1" />
       </joint>
@@ -528,5 +528,5 @@
          <origin xyz="-0.00025 -0.0007 -0.0775" rpy="0 0 0" />
          <axis xyz="1 0 0" />
-         <limit velocity="4.8" effort="1000" lower="-1.5804" upper="1.8201" />
+         <limit velocity="4.8" effort="1000" lower="-1.8201" upper="1.5804" />
          <dynamics damping="0.1" />
       </joint>

File: ffw_description/urdf/common/follower/ffw_follower_body.xacro (robot description, xacro)
@@ -304,5 +304,5 @@
          <origin xyz="0 0 -0.0885" rpy="0 0 0" />
          <axis xyz="1 0 0" />
-         <limit velocity="4.8" effort="1000" lower="-1.8201" upper="1.5804" />
+         <limit velocity="4.8" effort="1000" lower="-1.5804" upper="1.8201" />
          <dynamics damping="0.1" />
       </joint>
@@ -531,5 +531,5 @@
          <origin xyz="0 0 -0.0885" rpy="0 0 0" />
          <axis xyz="1 0 0" />
-         <limit velocity="4.8" effort="1000" lower="-1.5804" upper="1.8201" />
+         <limit velocity="4.8" effort="1000" lower="-1.8201" upper="1.5804" />
          <dynamics damping="0.1" />
       </joint>

File: ffw_description/urdf/ffw_bg2_rev4_follower/ffw_bg2_follower.urdf (robot description, URDF)
Before this commit: robot ffw_bg2_follower, 41 links, 40 joints
Joints:
- joint arm_l_joint7: limit lower=-1.8201 upper=1.5804 effort=1000 velocity=4.8 -> lower=-1.5804 upper=1.8201 effort=1000 velocity=4.8
- joint arm_r_joint7: limit lower=-1.5804 upper=1.8201 effort=1000 velocity=4.8 -> lower=-1.8201 upper=1.5804 effort=1000 velocity=4.8

File: ffw_description/urdf/ffw_f1_follower/ffw_f1_follower.urdf (robot description, URDF)
Before this commit: robot ffw_f1_follower, 37 links, 36 joints
Joints:
- joint arm_l_joint7: limit lower=-1.8201 upper=1.5804 effort=1000 velocity=4.8 -> lower=-1.5804 upper=1.8201 effort=1000 velocity=4.8
- joint arm_r_joint7: limit lower=-1.5804 upper=1.8201 effort=1000 velocity=4.8 -> lower=-1.8201 upper=1.5804 effort=1000 velocity=4.8

File: ffw_description/urdf/ffw_f2_follower/ffw_f2_follower.urdf (robot description, URDF)
Before this commit: robot ffw_f2_follower, 46 links, 45 joints
Joints:
- joint arm_l_joint7: limit lower=-1.8201 upper=1.5804 effort=1000 velocity=4.8 -> lower=-1.5804 upper=1.8201 effort=1000 velocity=4.8
- joint arm_r_joint7: limit lower=-1.5804 upper=1.8201 effort=1000 velocity=4.8 -> lower=-1.8201 upper=1.5804 effort=1000 velocity=4.8

File: ffw_description/urdf/ffw_sg2_rev1_follower/ffw_sg2_follower.urdf (robot description, URDF)
Before this commit: robot ffw_sg2_follower, 50 links, 49 joints
Joints:
- joint arm_l_joint7: limit lower=-1.8201 upper=1.5804 effort=1000 velocity=4.8 -> lower=-1.5804 upper=1.8201 effort=1000 velocity=4.8
- joint arm_r_joint7: limit lower=-1.5804 upper=1.8201 effort=1000 velocity=4.8 -> lower=-1.8201 upper=1.5804 effort=1000 velocity=4.8

File: ffw_description/urdf/ffw_sh5_rev1_follower/ffw_sh5_follower.urdf (robot description, URDF)
Before this commit: robot ffw_sh5_follower, 92 links, 91 joints
Joints:
- joint arm_l_joint7: limit lower=-1.8201 upper=1.5804 effort=1000 velocity=4.8 -> lower=-1.5804 upper=1.8201 effort=1000 velocity=4.8
- joint arm_r_joint7: limit lower=-1.5804 upper=1.8201 effort=1000 velocity=4.8 -> lower=-1.8201 upper=1.5804 effort=1000 velocity=4.8
