Commit message: refactor(ffw_description): modularize follower ros2_control by component
Signed-off-by: cmk-robotis <cmk@robotis.com>

File: ffw_description/ros2_control/follower/body/ffw.ros2_control.xacro (robot description, xacro)
@@ -1,34 +1,6 @@
 <?xml version="1.0"?>
 <robot xmlns:xacro="http://www.ros.org/wiki/xacro">
-  <xacro:macro name="ffw_sg2_follower_system" params="use_sim:=^|false use_mock_hardware:=^|false mock_sensor_commands:=^|false">
-    <ros2_control name="ffw_sg2_follower" type="system" is_async="true">
-      <xacro:if value="$(arg use_sim)">
-        <hardware>
-          <plugin>gz_ros2_control/GazeboSimSystem</plugin>
-        </hardware>
-      </xacro:if>
-      <xacro:unless value="$(arg use_sim)">
-        <hardware>
-          <xacro:if value="${use_mock_hardware}">
-            <plugin>mock_components/GenericSystem</plugin>
-            <param name="mock_sensor_commands">${mock_sensor_commands}</param>
-            <param name="state_following_offset">0.0</param>
-          </xacro:if>
-          <xacro:unless value="${use_mock_hardware}">
-            <plugin>dynamixel_hardware_interface/DynamixelHardware</plugin>
-            <param name="port_name">/dev/follower</param>
-            <param name="baud_rate">4000000</param>
-            <param name="dynamixel_model_folder">/param/dxl_model</param>
-            <param name="number_of_joints">22</param>
-            <param name="number_of_transmissions">22</param>
-            <param name="disable_torque_at_init">true</param>
-            <param name="dynamixel_state_pub_msg_name">ffw_follower/dxl_state</param>
-            <param name="get_dynamixel_data_srv_name">ffw_follower/get_dxl_data</param>
-            <param name="set_dynamixel_data_srv_name">ffw_follower/set_dxl_data</param>
-            <param name="reboot_dxl_srv_name">ffw_follower/reboot_dxl</param>
-            <param name="set_dxl_torque_srv_name">dynamixel_hardware_interface/set_dxl_torque</param>
-          </xacro:unless>
-        </hardware>
-      </xacro:unless>
+  <xacro:property name="follower_body_joint_count" value="17" />
+  <xacro:macro name="follower_body_joints">
       <joint name="arm_r_joint1">
         <command_interface name="position"/>
@@ -73,10 +45,4 @@
         <state_interface name="effort"/>
       </joint>
-      <joint name="gripper_r_joint1">
-        <command_interface name="position"/>
-        <state_interface name="position"/>
-        <state_interface name="velocity"/>
-        <state_interface name="effort"/>
-      </joint>
       <joint name="arm_l_joint1">
         <command_interface name="position"/>
@@ -121,10 +87,4 @@
         <state_interface name="effort"/>
       </joint>
-      <joint name="gripper_l_joint1">
-        <command_interface name="position"/>
-        <state_interface name="position"/>
-        <state_interface name="velocity"/>
-        <state_interface name="effort"/>
-      </joint>
       <joint name="lift_joint">
         <command_interface name="position"/>
@@ -140,22 +100,4 @@
       </joint>
       <joint name="head_joint2">
-        <command_interface name="position"/>
-        <state_interface name="position"/>
-        <state_interface name="velocity"/>
-        <state_interface name="effort"/>
-      </joint>
-      <joint name="left_wheel_steer">
-        <command_interface name="position"/>
-        <state_interface name="position"/>
-        <state_interface name="velocity"/>
-        <state_interface name="effort"/>
-      </joint>
-      <joint name="right_wheel_steer">
-        <command_interface name="position"/>
-        <state_interface name="position"/>
-        <state_interface name="velocity"/>
-        <state_interface name="effort"/>
-      </joint>
-      <joint name="rear_wheel_steer">
         <command_interface name="position"/>
         <state_interface name="position"/>
@@ -328,17 +270,4 @@
         <param name="Min Position Limit">-175979</param>
       </gpio>
-      <gpio name="dxl8">
-        <param name="type">dxl</param>
-        <param name="ID">8</param>
-        <command_interface name="Goal Position"/>
-        <state_interface name="Present Position"/>
-        <state_interface name="Present Velocity"/>
-        <state_interface name="Present Current"/>
-        <state_interface name="Hardware Error Status"/>
-        <param name="Operating Mode">5</param>
-        <param name="Return Delay Time">0</param>
-        <param name="Profile Velocity">0</param>
-        <param name="Profile Acceleration">0</param>
-      </gpio>
       <!-- LEFT ARM -->
       <gpio name="dxl31">
@@ -504,17 +433,4 @@
         <param name="Max Position Limit">175979</param>
         <param name="Min Position Limit">-152804</param>
-      </gpio>
-      <gpio name="dxl38">
-        <param name="type">dxl</param>
-        <param name="ID">38</param>
-        <command_interface name="Goal Position"/>
-        <state_interface name="Present Position"/>
-        <state_interface name="Present Velocity"/>
-        <state_interface name="Present Current"/>
-        <state_interface name="Hardware Error Status"/>
-        <param name="Operating Mode">5</param>
-        <param name="Return Delay Time">0</param>
-        <param name="Profile Velocity">0</param>
-        <param name="Profile Acceleration">0</param>
       </gpio>
       <!-- LIFT -->
@@ -592,65 +508,4 @@
         <param name="Feedforward 2nd Gain">20</param>
       </gpio>
-      <!-- LEFT WHEEL -->
-      <gpio name="dxl101">
-        <param name="type">dxl</param>
-        <param name="ID">101</param>
-        <command_interface name="Goal Position"/>
-        <state_interface name="Present Position"/>
-        <state_interface name="Present Velocity"/>
-        <state_interface name="Present Current"/>
-        <state_interface name="Error Code"/>
-        <param name="Drive Mode">5</param>
-        <param name="Operating Mode">3</param>
-        <param name="Velocity Limit">12592</param>
-        <param name="Acceleration Limit">125920</param>
-        <param name="Min Position Limit">-1572864</param>
-        <param name="Max Position Limit">1572864</param>
-        <param name="Return Delay Time">0</param>
-        <param name="Profile Velocity">12592</param>
-        <param name="Profile Acceleration Time">500</param>
-        <param name="Profile Time">1000</param>
-      </gpio>
-      <!-- RIGHT WHEEL -->
-      <gpio name="dxl103">
-        <param name="type">dxl</param>
-        <param name="ID">103</param>
-        <command_interface name="Goal Position"/>
-        <state_interface name="Present Position"/>
-        <state_interface name="Present Velocity"/>
-        <state_interface name="Present Current"/>
-        <state_interface name="Error Code"/>
-        <param name="Drive Mode">5</param>
-        <param name="Operating Mode">3</param>
-        <param name="Velocity Limit">12592</param>
-        <param name="Acceleration Limit">125920</param>
-        <param name="Min Position Limit">-1572864</param>
-        <param name="Max Position Limit">1572864</param>
-        <param name="Return Delay Time">0</param>
-        <param name="Profile Velocity">12592</param>
-        <param name="Profile Acceleration Time">500</param>
-        <param name="Profile Time">1000</param>
-      </gpio>
-      <!-- REAR WHEEL -->
-      <gpio name="dxl105">
-        <param name="type">dxl</param>
-        <param name="ID">105</param>
-        <command_interface name="Goal Position"/>
-        <state_interface name="Present Position"/>
-        <state_interface name="Present Velocity"/>
-        <state_interface name="Present Current"/>
-        <state_interface name="Error Code"/>
-        <param name="Drive Mode">5</param>
-        <param name="Operating Mode">3</param>
-        <param name="Velocity Limit">12592</param>
-        <param name="Acceleration Limit">125920</param>
-        <param name="Min Position Limit">-1572864</param>
-        <param name="Max Position Limit">1572864</param>
-        <param name="Return Delay Time">0</param>
-        <param name="Profile Velocity">12592</param>
-        <param name="Profile Acceleration Time">500</param>
-        <param name="Profile Time">1000</param>
-      </gpio>
-    </ros2_control>
   </xacro:macro>
 </robot>

File: ffw_description/ros2_control/follower/body/ffw_f.ros2_control.xacro (robot description, xacro)
@@ -1,34 +1,6 @@
 <?xml version="1.0"?>
 <robot xmlns:xacro="http://www.ros.org/wiki/xacro">
-  <xacro:macro name="ffw_f2_follower_system" params="use_sim:=^|false use_mock_hardware:=^|false mock_sensor_commands:=^|false">
-    <ros2_control name="ffw_f2_follower" type="system" is_async="true">
-      <xacro:if value="$(arg use_sim)">
-        <hardware>
-          <plugin>gz_ros2_control/GazeboSimSystem</plugin>
-        </hardware>
-      </xacro:if>
-      <xacro:unless value="$(arg use_sim)">
-        <hardware>
-          <xacro:if value="${use_mock_hardware}">
-            <plugin>mock_components/GenericSystem</plugin>
-            <param name="mock_sensor_commands">${mock_sensor_commands}</param>
-            <param name="state_following_offset">0.0</param>
-          </xacro:if>
-          <xacro:unless value="${use_mock_hardware}">
-            <plugin>dynamixel_hardware_interface/DynamixelHardware</plugin>
-            <param name="port_name">/dev/follower</param>
-            <param name="baud_rate">4000000</param>
-            <param name="dynamixel_model_folder">/param/dxl_model</param>
-            <param name="number_of_joints">22</param>
-            <param name="number_of_transmissions">22</param>
-            <param name="disable_torque_at_init">true</param>
-            <param name="dynamixel_state_pub_msg_name">ffw_follower/dxl_state</param>
-            <param name="get_dynamixel_data_srv_name">ffw_follower/get_dxl_data</param>
-            <param name="set_dynamixel_data_srv_name">ffw_follower/set_dxl_data</param>
-            <param name="reboot_dxl_srv_name">ffw_follower/reboot_dxl</param>
-            <param name="set_dxl_torque_srv_name">dynamixel_hardware_interface/set_dxl_torque</param>
-          </xacro:unless>
-        </hardware>
-      </xacro:unless>
+  <xacro:property name="follower_body_joint_count" value="17" />
+  <xacro:macro name="follower_body_joints">
       <joint name="arm_r_joint1">
         <command_interface name="position"/>
@@ -73,10 +45,4 @@
         <state_interface name="effort"/>
       </joint>
-      <joint name="gripper_r_joint1">
-        <command_interface name="position"/>
-        <state_interface name="position"/>
-        <state_interface name="velocity"/>
-        <state_interface name="effort"/>
-      </joint>
       <joint name="arm_l_joint1">
         <command_interface name="position"/>
@@ -121,10 +87,4 @@
         <state_interface name="effort"/>
       </joint>
-      <joint name="gripper_l_joint1">
-        <command_interface name="position"/>
-        <state_interface name="position"/>
-        <state_interface name="velocity"/>
-        <state_interface name="effort"/>
-      </joint>
       <joint name="lift_joint">
         <command_interface name="position"/>
@@ -140,22 +100,4 @@
       </joint>
       <joint name="head_joint2">
-        <command_interface name="position"/>
-        <state_interface name="position"/>
-        <state_interface name="velocity"/>
-        <state_interface name="effort"/>
-      </joint>
-      <joint name="left_wheel_steer">
-        <command_interface name="position"/>
-        <state_interface name="position"/>
-        <state_interface name="velocity"/>
-        <state_interface name="effort"/>
-      </joint>
-      <joint name="right_wheel_steer">
-        <command_interface name="position"/>
-        <state_interface name="position"/>
-        <state_interface name="velocity"/>
-        <state_interface name="effort"/>
-      </joint>
-      <joint name="rear_wheel_steer">
         <command_interface name="position"/>
         <state_interface name="position"/>
@@ -328,17 +270,4 @@
         <param name="Min Position Limit">-175979</param>
       </gpio>
-      <gpio name="dxl8">
-        <param name="type">dxl</param>
-        <param name="ID">8</param>
-        <command_interface name="Goal Position"/>
-        <state_interface name="Present Position"/>
-        <state_interface name="Present Velocity"/>
-        <state_interface name="Present Current"/>
-        <state_interface name="Hardware Error Status"/>
-        <param name="Operating Mode">5</param>
-        <param name="Return Delay Time">0</param>
-        <param name="Profile Velocity">0</param>
-        <param name="Profile Acceleration">0</param>
-      </gpio>
       <!-- LEFT ARM -->
       <gpio name="dxl31">
@@ -505,17 +434,4 @@
         <param name="Min Position Limit">-152804</param>
       </gpio>
-      <gpio name="dxl38">
-        <param name="type">dxl</param>
-        <param name="ID">38</param>
-        <command_interface name="Goal Position"/>
-        <state_interface name="Present Position"/>
-        <state_interface name="Present Velocity"/>
-        <state_interface name="Present Current"/>
-        <state_interface name="Hardware Error Status"/>
-        <param name="Operating Mode">5</param>
-        <param name="Return Delay Time">0</param>
-        <param name="Profile Velocity">0</param>
-        <param name="Profile Acceleration">0</param>
-      </gpio>
       <!-- LIFT -->
       <gpio name="dxl81">
@@ -563,5 +479,5 @@
         <param name="Profile Velocity">100</param>
         <param name="Profile Acceleration">50</param>
-        <param name="Max Position Limit">2500</param>
+        <param name="Max Position Limit">2560</param>
         <param name="Min Position Limit">1896</param>
         <param name="Position P Gain">1600</param>
@@ -592,68 +508,4 @@
         <param name="Feedforward 2nd Gain">20</param>
       </gpio>
-      <!-- LEFT WHEEL -->
-      <gpio name="dxl101">
-        <param name="type">dxl</param>
-        <param name="ID">101</param>
-        <command_interface name="Goal Position"/>
-        <state_interface name="Present Position"/>
-        <state_interface name="Present Velocity"/>
-        <state_interface name="Present Current"/>
-        <state_interface name="Error Code"/>
-        <param name="Drive Mode">5</param>
-        <param name="Operating Mode">3</param>
-        <param name="Velocity Limit">12592</param>
-        <param name="Acceleration Limit">125920</param>
-        <param name="Min Position Limit">-1572864</param>
-        <param name="Max Position Limit">1572864</param>
-        <param name="Acceleration Limit">1010</param>
-        <param name="Return Delay Time">0</param>
-        <param name="Profile Velocity">12592</param>
-        <param name="Profile Acceleration Time">500</param>
-        <param name="Profile Time">1000</param>
-      </gpio>
-      <!-- RIGHT WHEEL -->
-      <gpio name="dxl103">
-        <param name="type">dxl</param>
-        <param name="ID">103</param>
-        <command_interface name="Goal Position"/>
-        <state_interface name="Present Position"/>
-        <state_interface name="Present Velocity"/>
-        <state_interface name="Present Current"/>
-        <state_interface name="Error Code"/>
-        <param name="Drive Mode">5</param>
-        <param name="Operating Mode">3</param>
-        <param name="Velocity Limit">12592</param>
-        <param name="Acceleration Limit">125920</param>
-        <param name="Min Position Limit">-1572864</param>
-        <param name="Max Position Limit">1572864</param>
-        <param name="Acceleration Limit">1010</param>
-        <param name="Return Delay Time">0</param>
-        <param name="Profile Velocity">12592</param>
-        <param name="Profile Acceleration Time">500</param>
-        <param name="Profile Time">1000</param>
-      </gpio>
-      <!-- REAR WHEEL -->
-      <gpio name="dxl105">
-        <param name="type">dxl</param>
-        <param name="ID">105</param>
-        <command_interface name="Goal Position"/>
-        <state_interface name="Present Position"/>
-        <state_interface name="Present Velocity"/>
-        <state_interface name="Present Current"/>
-        <state_interface name="Error Code"/>
-        <param name="Drive Mode">5</param>
-        <param name="Operating Mode">3</param>
-        <param name="Velocity Limit">12592</param>
-        <param name="Acceleration Limit">125920</param>
-        <param name="Min Position Limit">-1572864</param>
-        <param name="Max Position Limit">1572864</param>
-        <param name="Acceleration Limit">1010</param>
-        <param name="Return Delay Time">0</param>
-        <param name="Profile Velocity">12592</param>
-        <param name="Profile Acceleration Time">500</param>
-        <param name="Profile Time">1000</param>
-      </gpio>
-    </ros2_control>
   </xacro:macro>
 </robot>

File: ffw_description/ros2_control/follower/ffw_follower.ros2_control.xacro (robot description, xacro)
@@ -1,9 +1,12 @@
 <?xml version="1.0"?>
 <robot xmlns:xacro="http://www.ros.org/wiki/xacro">
-  <xacro:include filename="$(find ffw_description)/ros2_control/ffw_sh5_rev1_follower/ffw_sh5_follower.joints.xacro" />
-  <xacro:include filename="$(find robotis_hand_description)/ros2_control/hx5_d20_rev2/hx5_d20_left.joints.xacro" />
-  <xacro:include filename="$(find robotis_hand_description)/ros2_control/hx5_d20_rev2/hx5_d20_right.joints.xacro" />
-  <xacro:macro name="ffw_sh5_follower_system" params="use_sim:=^|false use_mock_hardware:=^|false mock_sensor_commands:=^|false">
-    <ros2_control name="ffw_sh5_follower" type="system" is_async="true">
+  <xacro:include filename="$(find ffw_description)/ros2_control/follower/body/${robot_config['body']}.ros2_control.xacro" />
+  <xacro:include filename="$(find ffw_description)/ros2_control/follower/base/${robot_config['base']}.ros2_control.xacro" />
+  <xacro:include filename="$(find ffw_description)/ros2_control/follower/gripper/${robot_config['gripper']}.ros2_control.xacro" />
+  <xacro:macro name="follower_ros2_control"
+      params="use_sim use_mock_hardware mock_sensor_commands">
+    <xacro:property name="follower_joint_count"
+        value="${follower_body_joint_count + follower_base_steering_joint_count + follower_gripper_joint_count}" />
+    <ros2_control name="ffw_follower" type="system" is_async="true">
       <xacro:if value="${use_sim}">
         <hardware>
@@ -23,6 +26,6 @@
             <param name="baud_rate">4000000</param>
             <param name="dynamixel_model_folder">/param/dxl_model</param>
-            <param name="number_of_joints">60</param>
-            <param name="number_of_transmissions">60</param>
+            <param name="number_of_joints">${follower_joint_count}</param>
+            <param name="number_of_transmissions">${follower_joint_count}</param>
             <param name="disable_torque_at_init">true</param>
             <param name="dynamixel_state_pub_msg_name">ffw_follower/dxl_state</param>
@@ -34,8 +37,16 @@
         </hardware>
       </xacro:unless>
-      <xacro:hx5_right_joints/>
-      <xacro:hx5_left_joints/>
-      <xacro:ffw_sh5_follower_joints/>
+      <xacro:follower_body_joints />
+      <xacro:follower_gripper_joints />
+      <xacro:follower_base_steering_joints />
     </ros2_control>
+    <xacro:follower_base_drive_system
+        use_sim="${use_sim}"
+        use_mock_hardware="${use_mock_hardware}"
+        mock_sensor_commands="${mock_sensor_commands}" />
+    <xacro:follower_base_sensor_system
+        use_sim="${use_sim}"
+        use_mock_hardware="${use_mock_hardware}"
+        mock_sensor_commands="${mock_sensor_commands}" />
   </xacro:macro>
 </robot>

File: ffw_description/urdf/ffw_a3/ffw_a3.urdf.xacro (robot description, xacro)
@@ -5,5 +5,5 @@
   <xacro:arg name="mock_sensor_commands" default="false" />
   <xacro:arg name="prefix" default="" />
-  <xacro:include filename="$(find ffw_description)/urdf/common/leader/ffw_mini_leader_body.urdf.xacro" />
+  <xacro:include filename="$(find ffw_description)/urdf/leader/ffw_mini_leader_body.urdf.xacro" />
   <xacro:include filename="$(find ffw_description)/ros2_control/ffw_a3/ffw_a3.ros2_control.xacro" />
   <link name="world"/>

File: ffw_description/urdf/ffw_lg2_leader/ffw_lg2_leader.urdf.xacro (robot description, xacro)
@@ -5,5 +5,5 @@
   <xacro:arg name="mock_sensor_commands" default="false" />
   <xacro:arg name="prefix" default="" />
-  <xacro:include filename="$(find ffw_description)/urdf/common/leader/ffw_leader_body.urdf.xacro" />
+  <xacro:include filename="$(find ffw_description)/urdf/leader/ffw_leader_body.urdf.xacro" />
   <xacro:include filename="$(find ffw_description)/ros2_control/ffw_lg2_leader/ffw_lg2_leader_left.ros2_control.xacro" />
   <xacro:include filename="$(find ffw_description)/ros2_control/ffw_lg2_leader/ffw_lg2_leader_right.ros2_control.xacro" />

File: ffw_description/urdf/ffw_lg2_mini_leader/ffw_lg2_mini_leader.urdf.xacro (robot description, xacro)
@@ -5,5 +5,5 @@
   <xacro:arg name="mock_sensor_commands" default="false" />
   <xacro:arg name="prefix" default="" />
-  <xacro:include filename="$(find ffw_description)/urdf/common/leader/ffw_leader_body.urdf.xacro" />
+  <xacro:include filename="$(find ffw_description)/urdf/leader/ffw_leader_body.urdf.xacro" />
   <xacro:include filename="$(find ffw_description)/ros2_control/ffw_lg2_mini_leader/ffw_lg2_mini_leader_left.ros2_control.xacro" />
   <xacro:include filename="$(find ffw_description)/ros2_control/ffw_lg2_mini_leader/ffw_lg2_mini_leader_right.ros2_control.xacro" />

File: ffw_description/urdf/ffw_lg2_rev2_leader/ffw_lg2_rev2_leader.urdf.xacro (robot description, xacro)
@@ -5,5 +5,5 @@
   <xacro:arg name="mock_sensor_commands" default="false" />
   <xacro:arg name="prefix" default="" />
-  <xacro:include filename="$(find ffw_description)/urdf/common/leader/ffw_leader_body.urdf.xacro" />
+  <xacro:include filename="$(find ffw_description)/urdf/leader/ffw_leader_body.urdf.xacro" />
   <xacro:include filename="$(find ffw_description)/ros2_control/ffw_lg2_rev2_leader/ffw_lg2_rev2_leader_left.ros2_control.xacro" />
   <xacro:include filename="$(find ffw_description)/ros2_control/ffw_lg2_rev2_leader/ffw_lg2_rev2_leader_right.ros2_control.xacro" />
