Commit message: Update BH5 URDF
Signed-off-by: Hyunwoo Nam <nhw@robotis.com>

File: ffw_description/ros2_control/ffw_bh5_rev1_follower/ffw_bh5_follower.ros2_control.xacro (robot description, xacro)
@@ -1,4 +1,7 @@
 <?xml version="1.0"?>
 <robot xmlns:xacro="http://www.ros.org/wiki/xacro">
+  <xacro:include filename="$(find ffw_description)/ros2_control/$(arg model)/ffw_bh5_follower.joints.xacro" />
+  <xacro:include filename="$(find robotis_hand_description)/ros2_control/hx5_d20_rev2/hx5_d20_left.joints.xacro" />
+  <xacro:include filename="$(find robotis_hand_description)/ros2_control/hx5_d20_rev2/hx5_d20_right.joints.xacro" />
   <xacro:macro name="ffw_bh5_follower_system" params="use_sim:=^|false use_mock_hardware:=^|false mock_sensor_commands:=^|false">
     <ros2_control name="ffw_bh5_follower" type="system" is_async="true">
@@ -31,2701 +34,7 @@
         </hardware>
       </xacro:unless>
-      <joint name="finger_r_joint1">
-        <command_interface name="position"/>
-        <command_interface name="effort"/>
-        <state_interface name="position"/>
-        <state_interface name="velocity"/>
-        <state_interface name="effort"/>
-      </joint>
-      <joint name="finger_r_joint2">
-        <command_interface name="position"/>
-        <command_interface name="effort"/>
-        <state_interface name="position"/>
-        <state_interface name="velocity"/>
-        <state_interface name="effort"/>
-      </joint>
-      <joint name="finger_r_joint3">
-        <command_interface name="position"/>
-        <command_interface name="effort"/>
-        <state_interface name="position"/>
-        <state_interface name="velocity"/>
-        <state_interface name="effort"/>
-      </joint>
-      <joint name="finger_r_joint4">
-        <command_interface name="position"/>
-        <command_interface name="effort"/>
-        <state_interface name="position"/>
-        <state_interface name="velocity"/>
-        <state_interface name="effort"/>
-      </joint>
-      <sensor name="finger_r_sensor1">
-        <state_interface name="Present Pressure 1"/>
-        <state_interface name="Present Pressure 2"/>
-        <state_interface name="Present Pressure 3"/>
-        <state_interface name="Present Pressure 4"/>
-        <state_interface name="Present Pressure 5"/>
-        <state_interface name="Present Pressure 6"/>
-        <state_interface name="Present Pressure 7"/>
-        <state_interface name="Present Pressure 8"/>
-        <state_interface name="Present Pressure 9"/>
-      </sensor>
-      <joint name="finger_r_joint5">
-        <command_interface name="position"/>
-        <command_interface name="effort"/>
-        <state_interface name="position"/>
-        <state_interface name="velocity"/>
-        <state_interface name="effort"/>
-      </joint>
-      <joint name="finger_r_joint6">
-        <command_interface name="position"/>
-        <command_interface name="effort"/>
-        <state_interface name="position"/>
-        <state_interface name="velocity"/>
-        <state_interface name="effort"/>
-      </joint>
-      <joint name="finger_r_joint7">
-        <command_interface name="position"/>
-        <command_interface name="effort"/>
-        <state_interface name="position"/>
-        <state_interface name="velocity"/>
-        <state_interface name="effort"/>
-      </joint>
-      <joint name="finger_r_joint8">
-        <command_interface name="position"/>
-        <command_interface name="effort"/>
-        <state_interface name="position"/>
-        <state_interface name="velocity"/>
-        <state_interface name="effort"/>
-      </joint>
-      <sensor name="finger_r_sensor2">
-        <state_interface name="Present Pressure 1"/>
-        <state_interface name="Present Pressure 2"/>
-        <state_interface name="Present Pressure 3"/>
-        <state_interface name="Present Pressure 4"/>
-        <state_interface name="Present Pressure 5"/>
-        <state_interface name="Present Pressure 6"/>
-        <state_interface name="Present Pressure 7"/>
-        <state_interface name="Present Pressure 8"/>
-        <state_interface name="Present Pressure 9"/>
-      </sensor>
-      <joint name="finger_r_joint9">
-        <command_interface name="position"/>
-        <command_interface name="effort"/>
-        <state_interface name="position"/>
-        <state_interface name="velocity"/>
-        <state_interface name="effort"/>
-      </joint>
-      <joint name="finger_r_joint10">
-        <command_interface name="position"/>
-        <command_interface name="effort"/>
-        <state_interface name="position"/>
-        <state_interface name="velocity"/>
-        <state_interface name="effort"/>
-      </joint>
-      <joint name="finger_r_joint11">
-        <command_interface name="position"/>
-        <command_interface name="effort"/>
-        <state_interface name="position"/>
-        <state_interface name="velocity"/>
-        <state_interface name="effort"/>
-      </joint>
-      <joint name="finger_r_joint12">
-        <command_interface name="position"/>
-        <command_interface name="effort"/>
-        <state_interface name="position"/>
-        <state_interface name="velocity"/>
-        <state_interface name="effort"/>
-      </joint>
-      <sensor name="finger_r_sensor3">
-        <state_interface name="Present Pressure 1"/>
-        <state_interface name="Present Pressure 2"/>
-        <state_interface name="Present Pressure 3"/>
-        <state_interface name="Present Pressure 4"/>
-        <state_interface name="Present Pressure 5"/>
-        <state_interface name="Present Pressure 6"/>
-        <state_interface name="Present Pressure 7"/>
-        <state_interface name="Present Pressure 8"/>
-        <state_interface name="Present Pressure 9"/>
-      </sensor>
-      <joint name="finger_r_joint13">
-        <command_interface name="position"/>
-        <command_interface name="effort"/>
-        <state_interface name="position"/>
-        <state_interface name="velocity"/>
-        <state_interface name="effort"/>
-      </joint>
-      <joint name="finger_r_joint14">
-        <command_interface name="position"/>
-        <command_interface name="effort"/>
-        <state_interface name="position"/>
-        <state_interface name="velocity"/>
-        <state_interface name="effort"/>
-      </joint>
-      <joint name="finger_r_joint15">
-        <command_interface name="position"/>
-        <command_interface name="effort"/>
-        <state_interface name="position"/>
-        <state_interface name="velocity"/>
-        <state_interface name="effort"/>
-      </joint>
-      <joint name="finger_r_joint16">
-        <command_interface name="position"/>
-        <command_interface name="effort"/>
-        <state_interface name="position"/>
-        <state_interface name="velocity"/>
-        <state_interface name="effort"/>
-      </joint>
-      <sensor name="finger_r_sensor4">
-        <state_interface name="Present Pressure 1"/>
-        <state_interface name="Present Pressure 2"/>
-        <state_interface name="Present Pressure 3"/>
-        <state_interface name="Present Pressure 4"/>
-        <state_interface name="Present Pressure 5"/>
-        <state_interface name="Present Pressure 6"/>
-        <state_interface name="Present Pressure 7"/>
-        <state_interface name="Present Pressure 8"/>
-        <state_interface name="Present Pressure 9"/>
-      </sensor>
-      <joint name="finger_r_joint17">
-        <command_interface name="position"/>
-        <command_interface name="effort"/>
-        <state_interface name="position"/>
-        <state_interface name="velocity"/>
-        <state_interface name="effort"/>
-      </joint>
-      <joint name="finger_r_joint18">
-        <command_interface name="position"/>
-        <command_interface name="effort"/>
-        <state_interface name="position"/>
-        <state_interface name="velocity"/>
-        <state_interface name="effort"/>
-      </joint>
-      <joint name="finger_r_joint19">
-        <command_interface name="position"/>
-        <command_interface name="effort"/>
-        <state_interface name="position"/>
-        <state_interface name="velocity"/>
-        <state_interface name="effort"/>
-      </joint>
-      <joint name="finger_r_joint20">
-        <command_interface name="position"/>
-        <command_interface name="effort"/>
-        <state_interface name="position"/>
-        <state_interface name="velocity"/>
-        <state_interface name="effort"/>
-      </joint>
-      <sensor name="finger_r_sensor5">
-        <state_interface name="Present Pressure 1"/>
-        <state_interface name="Present Pressure 2"/>
-        <state_interface name="Present Pressure 3"/>
-        <state_interface name="Present Pressure 4"/>
-        <state_interface name="Present Pressure 5"/>
-        <state_interface name="Present Pressure 6"/>
-        <state_interface name="Present Pressure 7"/>
-        <state_interface name="Present Pressure 8"/>
-        <state_interface name="Present Pressure 9"/>
-      </sensor>
-      <joint name="arm_r_joint1">
-        <command_interface name="position"/>
-        <state_interface name="position"/>
-        <state_interface name="velocity"/>
-        <state_interface name="effort"/>
-      </joint>
-      <joint name="arm_r_joint2">
-        <command_interface name="position"/>
-        <state_interface name="position"/>
-        <state_interface name="velocity"/>
-        <state_interface name="effort"/>
-      </joint>
-      <joint name="arm_r_joint3">
-        <command_interface name="position"/>
-        <state_interface name="position"/>
-        <state_interface name="velocity"/>
-        <state_interface name="effort"/>
-      </joint>
-      <joint name="arm_r_joint4">
-        <command_interface name="position"/>
-        <state_interface name="position"/>
-        <state_interface name="velocity"/>
-        <state_interface name="effort"/>
-      </joint>
-      <joint name="arm_r_joint5">
-        <command_interface name="position"/>
-        <state_interface name="position"/>
-        <state_interface name="velocity"/>
-        <state_interface name="effort"/>
-      </joint>
-      <joint name="arm_r_joint6">
-        <command_interface name="position"/>
-        <state_interface name="position"/>
-        <state_interface name="velocity"/>
-        <state_interface name="effort"/>
-      </joint>
-      <joint name="arm_r_joint7">
-        <command_interface name="position"/>
-        <state_interface name="position"/>
-        <state_interface name="velocity"/>
-        <state_interface name="effort"/>
-      </joint>
-      <joint name="finger_l_joint1">
-        <command_interface name="position"/>
-        <command_interface name="effort"/>
-        <state_interface name="position"/>
-        <state_interface name="velocity"/>
-        <state_interface name="effort"/>
-      </joint>
-      <joint name="finger_l_joint2">
-        <command_interface name="position"/>
-        <command_interface name="effort"/>
-        <state_interface name="position"/>
-        <state_interface name="velocity"/>
-        <state_interface name="effort"/>
-      </joint>
-      <joint name="finger_l_joint3">
-        <command_interface name="position"/>
-        <command_interface name="effort"/>
-        <state_interface name="position"/>
-        <state_interface name="velocity"/>
-        <state_interface name="effort"/>
-      </joint>
-      <joint name="finger_l_joint4">
-        <command_interface name="position"/>
-        <command_interface name="effort"/>
-        <state_interface name="position"/>
-        <state_interface name="velocity"/>
-        <state_interface name="effort"/>
-      </joint>
-      <sensor name="finger_l_sensor1">
-        <state_interface name="Present Pressure 1"/>
-        <state_interface name="Present Pressure 2"/>
-        <state_interface name="Present Pressure 3"/>
-        <state_interface name="Present Pressure 4"/>
-        <state_interface name="Present Pressure 5"/>
-        <state_interface name="Present Pressure 6"/>
-        <state_interface name="Present Pressure 7"/>
-        <state_interface name="Present Pressure 8"/>
-        <state_interface name="Present Pressure 9"/>
-      </sensor>
-      <joint name="finger_l_joint5">
-        <command_interface name="position"/>
-        <command_interface name="effort"/>
-        <state_interface name="position"/>
-        <state_interface name="velocity"/>
-        <state_interface name="effort"/>
-      </joint>
-      <joint name="finger_l_joint6">
-        <command_interface name="position"/>
-        <command_interface name="effort"/>
-        <state_interface name="position"/>
-        <state_interface name="velocity"/>
-        <state_interface name="effort"/>
-      </joint>
-      <joint name="finger_l_joint7">
-        <command_interface name="position"/>
-        <command_interface name="effort"/>
-        <state_interface name="position"/>
-        <state_interface name="velocity"/>
-        <state_interface name="effort"/>
-      </joint>
-      <joint name="finger_l_joint8">
-        <command_interface name="position"/>
-        <command_interface name="effort"/>
-        <state_interface name="position"/>
-        <state_interface name="velocity"/>
-        <state_interface name="effort"/>
-      </joint>
-      <sensor name="finger_l_sensor2">
-        <state_interface name="Present Pressure 1"/>
-        <state_interface name="Present Pressure 2"/>
-        <state_interface name="Present Pressure 3"/>
-        <state_interface name="Present Pressure 4"/>
-        <state_interface name="Present Pressure 5"/>
-        <state_interface name="Present Pressure 6"/>
-        <state_interface name="Present Pressure 7"/>
-        <state_interface name="Present Pressure 8"/>
-        <state_interface name="Present Pressure 9"/>
-      </sensor>
-      <joint name="finger_l_joint9">
-        <command_interface name="position"/>
-        <command_interface name="effort"/>
-        <state_interface name="position"/>
-        <state_interface name="velocity"/>
-        <state_interface name="effort"/>
-      </joint>
-      <joint name="finger_l_joint10">
-        <command_interface name="position"/>
-        <command_interface name="effort"/>
-        <state_interface name="position"/>
-        <state_interface name="velocity"/>
-        <state_interface name="effort"/>
-      </joint>
-      <joint name="finger_l_joint11">
-        <command_interface name="position"/>
-        <command_interface name="effort"/>
-        <state_interface name="position"/>
-        <state_interface name="velocity"/>
-        <state_interface name="effort"/>
-      </joint>
-      <joint name="finger_l_joint12">
-        <command_interface name="position"/>
-        <command_interface name="effort"/>
-        <state_interface name="position"/>
-        <state_interface name="velocity"/>
-        <state_interface name="effort"/>
-      </joint>
-      <sensor name="finger_l_sensor3">
-        <state_interface name="Present Pressure 1"/>
-        <state_interface name="Present Pressure 2"/>
-        <state_interface name="Present Pressure 3"/>
-        <state_interface name="Present Pressure 4"/>
-        <state_interface name="Present Pressure 5"/>
-        <state_interface name="Present Pressure 6"/>
-        <state_interface name="Present Pressure 7"/>
-        <state_interface name="Present Pressure 8"/>
-        <state_interface name="Present Pressure 9"/>
-      </sensor>
-      <joint name="finger_l_joint13">
-        <command_interface name="position"/>
-        <command_interface name="effort"/>
-        <state_interface name="position"/>
-        <state_interface name="velocity"/>
-        <state_interface name="effort"/>
-      </joint>
-      <joint name="finger_l_joint14">
-        <command_interface name="position"/>
-        <command_interface name="effort"/>
-        <state_interface name="position"/>
-        <state_interface name="velocity"/>
-        <state_interface name="effort"/>
-      </joint>
-      <joint name="finger_l_joint15">
-        <command_interface name="position"/>
-        <command_interface name="effort"/>
-        <state_interface name="position"/>
-        <state_interface name="velocity"/>
-        <state_interface name="effort"/>
-      </joint>
-      <joint name="finger_l_joint16">
-        <command_interface name="position"/>
-        <command_interface name="effort"/>
-        <state_interface name="position"/>
-        <state_interface name="velocity"/>
-        <state_interface name="effort"/>
-      </joint>
-      <sensor name="finger_l_sensor4">
-        <state_interface name="Present Pressure 1"/>
-        <state_interface name="Present Pressure 2"/>
-        <state_interface name="Present Pressure 3"/>
-        <state_interface name="Present Pressure 4"/>
-        <state_interface name="Present Pressure 5"/>
-        <state_interface name="Present Pressure 6"/>
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
File: ffw_description/urdf/ffw_bh5_rev1_follower/ffw_bh5_follower.urdf.xacro (robot description, xacro)
@@ -10,9 +10,10 @@
   <xacro:arg name="ros2_control_type" default="ffw_bh5_follower" />
   <xacro:include filename="$(find ffw_description)/urdf/common/follower/ffw_follower_body.xacro" />
-  <xacro:include filename="$(find ffw_description)/urdf/common/hx5_d20/hx5_d20_left.urdf.xacro" />
-  <xacro:include filename="$(find ffw_description)/urdf/common/hx5_d20/hx5_d20_right.urdf.xacro" />
-  <!-- Reuse the proven BH5 upper-body ros2_control definition for BH5. -->
+  <xacro:include filename="$(find robotis_hand_description)/urdf/hx5_d20_rev2/hx5_d20_left.urdf.xacro" />
+  <xacro:include filename="$(find robotis_hand_description)/urdf/hx5_d20_rev2/hx5_d20_right.urdf.xacro" />
   <xacro:include filename="$(find ffw_description)/ros2_control/ffw_bh5_rev1_follower/ffw_bh5_follower.ros2_control.xacro" />
   <xacro:include filename="$(find ffw_description)/gazebo/$(arg model)/ffw_bh5_follower.gazebo.xacro" />
+  <xacro:include filename="$(find robotis_hand_description)/gazebo/hx5_d20/hx5_d20_left.gazebo.xacro" />
+  <xacro:include filename="$(find robotis_hand_description)/gazebo/hx5_d20/hx5_d20_right.gazebo.xacro" />
   <link name="world"/>
   <joint name="$(arg prefix)world_fixed" type="fixed">
@@ -48,10 +49,16 @@
     <origin xyz="0.0055 0 1.4316" rpy="0 0 0" />
   </xacro:ffw_follower_body>
-  <xacro:hx5_d20_left parent="$(arg prefix)arm_l_link7" prefix="$(arg prefix)">
+  <joint name="$(arg prefix)hx5_d20_left_joint" type="fixed">
+    <parent link="$(arg prefix)arm_l_link7"/>
+    <child link="$(arg prefix)hx5_d20_left_base"/>
     <origin xyz="0 0 -0.078" rpy="0 3.14159265359 1.5708"/>
-  </xacro:hx5_d20_left>
-  <xacro:hx5_d20_right parent="$(arg prefix)arm_r_link7" prefix="$(arg prefix)">
+  </joint>
+  <xacro:hx5_d20_left prefix="$(arg prefix)" />
+  <joint name="$(arg prefix)hx5_d20_right_joint" type="fixed">
+    <parent link="$(arg prefix)arm_r_link7"/>
+    <child link="$(arg prefix)hx5_d20_right_base"/>
     <origin xyz="0 0 -0.078" rpy="0 3.14159265359 -1.5708"/>
-  </xacro:hx5_d20_right>
+  </joint>
+  <xacro:hx5_d20_right prefix="$(arg prefix)" />
   <xacro:ffw_bh5_follower_system
     use_sim="$(arg use_sim)"
