Commit message: Fix a3 leader controller error
Signed-off-by: cmk-robotis <cmk@robotis.com>

File: ffw_description/ros2_control/ffw_a3/ffw_a3.ros2_control.xacro (robot description, xacro)
@@ -56,7 +56,6 @@
       </sensor>
       <joint name="gripper_l_joint1">
-        <command_interface name="effort"/>
-        <state_interface name="position"/>
-        <state_interface name="velocity"/>
+        <command_interface name="position"/>
+        <state_interface name="position"/>
       </joint>
       <joint name="arm_l_joint1">
@@ -87,7 +86,6 @@
       </sensor>
       <joint name="gripper_r_joint1">
-        <command_interface name="effort"/>
-        <state_interface name="position"/>
-        <state_interface name="velocity"/>
+        <command_interface name="position"/>
+        <state_interface name="position"/>
       </joint>
       <joint name="arm_r_joint1">
@@ -131,5 +129,5 @@
         <param name="Position D Gain">300</param>
         <param name="Current Limit">100</param>
-        <param name="Homing Offset">200</param>
+        <param name="Homing Offset">0</param>
       </gpio>
       <gpio name="dxl31">
@@ -215,5 +213,5 @@
         <param name="Position D Gain">300</param>
         <param name="Current Limit">100</param>
-        <param name="Homing Offset">-200</param>
+        <param name="Homing Offset">0</param>
       </gpio>
       <gpio name="dxl1">

File: ffw_description/urdf/follower/body/ffw_body.urdf.xacro (robot description, xacro)
@@ -42,5 +42,5 @@
          <origin xyz="0.049483 0 0.102130" rpy="0 0 0" />
          <axis xyz="0 1 0" />
-         <limit velocity="4.8" effort="1000" lower="-0.2317" upper="0.6951" />
+         <limit velocity="4.8" effort="1000" lower="-0.2317" upper="0.83" />
          <dynamics damping="0.1" />
       </joint>

File: ffw_description/urdf/follower/body/ffw_body_f.urdf.xacro (robot description, xacro)
@@ -42,5 +42,5 @@
          <origin xyz="0.102729 0 0.132803" rpy="0 0 0" />
          <axis xyz="0 1 0" />
-         <limit velocity="4.8" effort="1000" lower="-0.2317" upper="0.6951" />
+         <limit velocity="4.8" effort="1000" lower="-0.2317" upper="0.83" />
          <dynamics damping="0.1" />
       </joint>

Commit message: feat: add leader port detection to ffw_a3 launch
Signed-off-by: cmk-robotis <cmk@robotis.com>

File: ffw_description/ros2_control/ffw_a3/ffw_a3.ros2_control.xacro (robot description, xacro)
@@ -1,5 +1,5 @@
 <?xml version="1.0"?>
 <robot xmlns:xacro="http://www.ros.org/wiki/xacro">
-  <xacro:macro name="ffw_a3_system" params="use_sim:=^|false use_mock_hardware:=^|false mock_sensor_commands:=^|false">
+  <xacro:macro name="ffw_a3_system" params="use_sim:=^|false use_mock_hardware:=^|false mock_sensor_commands:=^|false port_name:=^|/dev/leader">
     <xacro:property name="initial_positions" value="${load_yaml(initial_positions_file)['initial_positions']}"/>
     <ros2_control name="ffw_a3" type="system" is_async="true">
@@ -18,5 +18,5 @@
           <xacro:unless value="${use_mock_hardware}">
             <plugin>dynamixel_hardware_interface/DynamixelHardware</plugin>
-            <param name="port_name">/dev/leader</param>
+            <param name="port_name">${port_name}</param>
             <param name="baud_rate">4000000</param>
             <param name="dynamixel_model_folder">/param/dxl_model</param>

File: ffw_description/urdf/ffw_a3/ffw_a3.urdf.xacro (robot description, xacro)
@@ -5,4 +5,5 @@
   <xacro:arg name="mock_sensor_commands" default="false" />
   <xacro:arg name="prefix" default="" />
+  <xacro:arg name="port_name" default="/dev/leader" />
   <xacro:include filename="$(find ffw_description)/urdf/leader/ffw_mini_leader_body.urdf.xacro" />
   <xacro:include filename="$(find ffw_description)/ros2_control/ffw_a3/ffw_a3.ros2_control.xacro" />
@@ -14,4 +15,5 @@
       use_sim="$(arg use_sim)"
       use_mock_hardware="$(arg use_mock_hardware)"
+      port_name="$(arg port_name)"
       mock_sensor_commands="$(arg mock_sensor_commands)" />
 </robot>
