Commit message: Added a2 urdf

File: ffw_description/urdf/common/leader/ffw_mini_leader_body.urdf.xacro (robot description, xacro)
@@ -2,11 +2,10 @@
 <robot xmlns:xacro="http://www.ros.org/wiki/xacro">
    <xacro:macro name="ffw_mini_leader_body" params="prefix parent *origin">
-      <xacro:property name="meshes_file_direction" value="package://ffw_description/meshes/ffw_lg2_rev3_leader" />
-      <joint name="${prefix}joint" type="prismatic">
+      <xacro:property name="meshes_file_direction" value="package://ffw_description/meshes/common/leader" />
+      <joint name="${prefix}joint" type="fixed">
          <parent link="${parent}"/>
          <child link="${prefix}arm_base_link" />
          <xacro:insert_block name="origin" />
          <axis xyz="0 0 1" />
-         <limit velocity="4.8" effort="1000" lower="0.0" upper="0.25" />
          <dynamics damping="0.1" />
       </joint>

Commit message: Updated a2 urdf and meshes

File: ffw_description/urdf/common/leader/ffw_mini_leader_body.urdf.xacro (robot description, xacro)
@@ -2,5 +2,5 @@
 <robot xmlns:xacro="http://www.ros.org/wiki/xacro">
    <xacro:macro name="ffw_mini_leader_body" params="prefix parent *origin">
-      <xacro:property name="meshes_file_direction" value="package://ffw_description/meshes/common/leader" />
+      <xacro:property name="meshes_file_direction" value="package://ffw_description/meshes/common/leader/a2" />
       <joint name="${prefix}joint" type="fixed">
          <parent link="${parent}"/>
@@ -27,13 +27,13 @@
          </collision>
          <inertial>
-            <origin xyz="0.0073855606 0.000013925213 -0.00031328687" rpy="0 0 0" />
-            <mass value="0.33009790" />
-            <inertia
-               ixx="0.0021452770"
-               ixy="-0.000000016680053"
-               ixz="-0.00000088143244"
-               iyy="0.00014049217"
-               iyz="0.00000012031854"
-               izz="0.0021934172" />
+            <origin xyz="1.0347495e-02  5.9413880e-05 -7.6051910e-04" rpy="0 0 0" />
+            <mass value="3.7813639e-01" />
+            <inertia
+               ixx="2.2075825e-03"
+               ixy="2.7587134e-07"
+               ixz="4.0606472e-06"
+               iyy="1.8920594e-04"
+               iyz="6.3038012e-08"
+               izz="2.2758983e-03" />
          </inertial>
       </link>
@@ -350,13 +350,13 @@
          </collision>
          <inertial>
-            <origin xyz="0.00031402977 -0.032879331 -0.000027429864" rpy="0 0 0" />
-            <mass value="0.026192376" />
-            <inertia
-               ixx="0.0000039979965"
-               ixy="0.000000010639622"
-               ixz="0.000000000022505889"
-               iyy="0.0000021593469"
-               iyz="0.0000000039430261"
-               izz="0.0000044607896" />
+            <origin xyz="3.1402977e-04 -3.2879331e-02 -2.7429864e-05" rpy="0 0 0" />
+            <mass value="2.6192376e-02" />
+            <inertia
+               ixx="3.9979965e-06"
+               ixy="1.0639622e-08"
+               ixz="2.2505889e-11"
+               iyy="2.1593469e-06"
+               iyz="3.9430261e-09"
+               izz="4.4607896e-06" />
          </inertial>
       </link>
@@ -386,13 +386,13 @@
          </collision>
          <inertial>
-            <origin xyz="0.00047440645 0.00050549060 -0.053005948" rpy="0 0 0" />
-            <mass value="0.049263777" />
-            <inertia
-               ixx="0.000045012579"
-               ixy="0.000000010933721"
-               ixz="0.00000031844474"
-               iyy="0.000048394473"
-               iyz="0.0000014801494"
-               izz="0.0000076982778" />
+            <origin xyz="5.2815896e-04  8.4254963e-04 -5.3432730e-02" rpy="0 0 0" />
+            <mass value="4.8908171e-02" />
+            <inertia
+               ixx="4.5540567e-05"
+               ixy="1.9786829e-08"
+               ixz="3.3082854e-07"
+               iyy="4.8853649e-05"
+               iyz="1.2884556e-06"
+               izz="7.7762219e-06" />
          </inertial>
       </link>
@@ -422,13 +422,13 @@
          </collision>
          <inertial>
-            <origin xyz="0.0044577228 -0.0039566353 -0.018293795" rpy="0 0 0" />
-            <mass value="0.055181999" />
-            <inertia
-               ixx="0.000023484710"
-               ixy="-0.0000010244284"
-               ixz="0.0000055436948"
-               iyy="0.000023065957"
-               iyz="0.0000029244542"
-               izz="0.0000094498947" />
+            <origin xyz="4.4279540e-03 -3.9794114e-03 -1.8251483e-02" rpy="0 0 0" />
+            <mass value="5.5538993e-02" />
+            <inertia
+               ixx="2.3569109e-05"
+               ixy="-1.0302491e-06"
+               ixz="5.5589832e-06"
+               iyy="2.3107503e-05"
+               iyz="2.9327276e-06"
+               izz="9.5533558e-06" />
          </inertial>
       </link>
@@ -458,13 +458,13 @@
          </collision>
          <inertial>
-            <origin xyz="-0.014359796 0.0012830993 -0.034672139" rpy="0 0 0" />
-            <mass value="0.040899967" />
-            <inertia
-               ixx="0.000022527545"
-               ixy="0.00000011623193"
-               ixz="-0.0000027613358"
-               iyy="0.000020374424"
-               iyz="0.0000011035415"
-               izz="0.0000081410810" />
+            <origin xyz="-1.4327210e-02  1.2848970e-03 -3.4625542e-02" rpy="0 0 0" />
+            <mass value="4.0932690e-02" />
+            <inertia
+               ixx="2.2633568e-05"
+               ixy="1.1551007e-07"
+               ixz="-2.8098147e-06"
+               iyy="2.0477488e-05"
+               iyz="1.1027614e-06"
+               izz="8.1858151e-06" />
          </inertial>
       </link>

Commit message: Modified a2 urdf inertials

File: ffw_description/urdf/common/leader/ffw_mini_leader_body.urdf.xacro (robot description, xacro)
@@ -63,13 +63,13 @@
          </collision>
          <inertial>
-            <origin xyz="0.00021402977 0.032879331 0.000027429864" rpy="0 0 0" />
-            <mass value="0.026192376" />
-            <inertia
-               ixx="0.0000039979965"
-               ixy="-0.000000010639622"
-               ixz="-0.000000000022505889"
-               iyy="0.0000021593469"
-               iyz="0.0000000039430261"
-               izz="0.0000044607896" />
+            <origin xyz="3.1402977e-04  3.2879331e-02  2.7429864e-05" rpy="0 0 0" />
+            <mass value="2.6192376e-02" />
+            <inertia
+               ixx="3.9979965e-06"
+               ixy="-1.0639622e-07"
+               ixz="-2.2505889e-11"
+               iyy="2.1593469e-06"
+               iyz="3.9430261e-09"
+               izz="4.4607896e-06" />
          </inertial>
       </link>
@@ -99,13 +99,13 @@
          </collision>
          <inertial>
-            <origin xyz="0.00036878960 -0.00047925236 -0.053011125" rpy="0 0 0" />
-            <mass value="0.049309095" />
-            <inertia
-               ixx="0.000044955210"
-               ixy="-0.0000000077712199"
-               ixz="0.00000031630287"
-               iyy="0.000048329957"
-               iyz="-0.0000015048615"
-               izz="0.0000077071863" />
+            <origin xyz="5.2188296e-04 -8.2173051e-04 -5.3407063e-02" rpy="0 0 0" />
+            <mass value="4.9006818e-02" />
+            <inertia
+               ixx="4.5563627e-05"
+               ixy="-1.6612287e-08"
+               ixz="3.2957186e-07"
+               iyy="4.8869230e-05"
+               iyz="-1.3039000e-06"
+               izz="7.7898213e-06" />
          </inertial>
       </link>
@@ -135,13 +135,13 @@
          </collision>
          <inertial>
-            <origin xyz="0.0043653496 0.0039566345 -0.018335049" rpy="0 0 0" />
-            <mass value="0.055181999" />
-            <inertia
-               ixx="0.000023490482"
-               ixy="0.0000010054524"
-               ixz="0.0000054999352"
-               iyy="0.000023055403"
-               iyz="-0.0000029236575"
-               izz="0.0000094335676" />
+            <origin xyz="4.4355318e-03  3.9794105e-03 -1.8269777e-02" rpy="0 0 0" />
+            <mass value="5.5538993e-02" />
+            <inertia
+               ixx="2.3595371e-05"
+               ixy="1.0112827e-06"
+               ixz="5.5208999e-06"
+               iyy="2.3117463e-05"
+               iyz="-2.9364202e-06"
+               izz="9.5370537e-06" />
          </inertial>
       </link>
@@ -171,13 +171,13 @@
          </collision>
          <inertial>
-            <origin xyz="-0.014378495 -0.0012413463 -0.034680174" rpy="0 0 0" />
-            <mass value="0.040992686" />
-            <inertia
-               ixx="0.000022551700"
-               ixy="-0.00000010396374"
-               ixz="-0.0000027636794"
-               iyy="0.000020383931"
-               iyz="-0.0000010927665"
-               izz="0.0000081674213" />
+            <origin xyz="-1.4345968e-02 -1.2431732e-03 -3.4633676e-02" rpy="0 0 0" />
+            <mass value="4.1025410e-02" />
+            <inertia
+               ixx="2.2657760e-05"
+               ixy="-1.0318482e-07"
+               ixz="-2.8122047e-06"
+               iyy="2.0487075e-05"
+               iyz="-1.0919062e-06"
+               izz="8.2122115e-06" />
          </inertial>
       </link>
@@ -207,13 +207,13 @@
          </collision>
          <inertial>
-            <origin xyz="0 0.0037848539 -0.018058013" rpy="0 0 0" />
-            <mass value="0.052704760" />
-            <inertia
-               ixx="0.000024222035"
-               ixy="-0.000000010247619"
-               ixz="-0.000000021364276"
-               iyy="0.000021227718"
-               iyz="-0.0000029349250"
-               izz="0.0000064055965" />
+            <origin xyz="0.0000000e+00  3.8292440e-03 -1.8018759e-02" rpy="0 0 0" />
+            <mass value="5.3343451e-02" />
+            <inertia
+               ixx="2.4359040e-05"
+               ixy="-1.0247646e-08"
+               ixz="-2.1364272e-08"
+               iyy="2.1273792e-05"
+               iyz="-2.9431209e-06"
+               izz="6.5911205e-06" />
          </inertial>
       </link>
@@ -243,13 +243,13 @@
          </collision>
          <inertial>
-            <origin xyz="0.00025734695 -0.000022479263 -0.027933324" rpy="0 0 0" />
-            <mass value="0.031961547" />
-            <inertia
-               ixx="0.0000080476878"
-               ixy="0.000000000063240356"
-               ixz="0.000000060814731"
-               iyy="0.0000076232281"
-               iyz="-0.000000010184417"
-               izz="0.0000035088531" />
+            <origin xyz="2.5655803e-04 -2.2409583e-05 -2.7826901e-02" rpy="0 0 0" />
+            <mass value="3.2059818e-02" />
+            <inertia
+               ixx="8.2117295e-06"
+               ixy="6.3818774e-11"
+               ixz="6.1690103e-08"
+               iyy="7.7657254e-06"
+               iyz="-1.0260980e-08"
+               izz="3.6178162e-06" />
          </inertial>
       </link>
@@ -279,13 +279,13 @@
          </collision>
          <inertial>
-            <origin xyz="-0.047767307 -0.0065309978 -0.086992041" rpy="0 0 0" />
-            <mass value="0.30390944" />
-            <inertia
-               ixx="0.00050134919"
-               ixy="0.000042309966"
-               ixz="0.000040549745"
-               iyy="0.00095578295"
-               iyz="-0.000058682543"
-               izz="0.00056175585" />
+            <origin xyz="-4.5917284e-02 -1.0476763e-02 -1.0251170e-01" rpy="0 0 0" />
+            <mass value="2.3810068e-01" />
+            <inertia
+               ixx="4.8502443e-04"
+               ixy="4.8822587e-06"
+               ixz="-2.7728350e-05"
+               iyy="6.8976363e-04"
+               iyz="-7.9136483e-05"
+               izz="3.2999961e-04" />
          </inertial>
       </link>
@@ -314,13 +314,13 @@
          </collision>
          <inertial>
-            <origin xyz="-0.0088471289 -0.000056545778 0.0063502762" rpy="0 0 0" />
-            <mass value="0.0060222456" />
-            <inertia
-               ixx="0.00000057813523"
-               ixy="0.0000000030127359"
-               ixz="0.00000023215673"
-               iyy="0.0000012235266"
-               iyz="-0.0000000021624756"
-               izz="0.00000073651828" />
+            <origin xyz="-8.6845430e-03 -3.1215916e-04  6.2417800e-03" rpy="0 0 0" />
+            <mass value="3.4935532e-03" />
+            <inertia
+               ixx="3.1731773e-07"
+               ixy="9.4708822e-09"
+               ixz="1.3547192e-07"
+               iyy="7.0503093e-07"
+               iyz="-6.8069391e-09"
+               izz="4.0910624e-07" />
          </inertial>
       </link>
@@ -494,13 +494,13 @@
          </collision>
          <inertial>
-            <origin xyz="0 -0.0037848539 -0.018058013" rpy="0 0 0" />
-            <mass value="0.052704760" />
-            <inertia
-               ixx="0.000024222035"
-               ixy="-0.000000010247618"
-               ixz="0.000000021364273"
-               iyy="0.000021227718"
-               iyz="0.0000029349250"
-               izz="0.0000064055965" />
+            <origin xyz="0.0000000e+00 -3.8292440e-03 -1.8018759e-02" rpy="0 0 0" />
+            <mass value="5.3343451e-02" />
+            <inertia
+               ixx="2.4359040e-05"
+               ixy="-1.0247645e-07"
+               ixz="2.1364269e-08"
+               iyy="2.1273792e-05"
+               iyz="2.9431209e-06"
+               izz="6.5911205e-06" />
          </inertial>
       </link>
@@ -530,13 +530,13 @@
          </collision>
          <inertial>
-            <origin xyz="0.00025734695 -0.000022479263 -0.027933324" rpy="0 0 0" />
-            <mass value="0.031961547" />
-            <inertia
-               ixx="0.0000080476878"
-               ixy="0.000000000063240356"
-               ixz="0.000000060814731"
-               iyy="0.0000076232281"
-               iyz="-0.000000010184417"
-               izz="0.0000035088531" />
+            <origin xyz="2.5655803e-04 -2.2409583e-05 -2.7826901e-02" rpy="0 0 0" />
+            <mass value="3.2059818e-02" />
+            <inertia
+               ixx="8.2117295e-06"
+               ixy="6.3818774e-11"
+               ixz="6.1690103e-08"
+               iyy="7.7657254e-06"
+               iyz="-1.0260980e-08"
+               izz="3.6178162e-06" />
          </inertial>
       </link>
@@ -566,13 +566,13 @@
          </collision>
          <inertial>
-            <origin xyz="-0.047110855 0.0067030274 -0.086068978" rpy="0 0 0" />
-            <mass value="0.30067384" />
-            <inertia
-               ixx="0.00048869771"
-               ixy="-0.000040597374"
-               ixz="0.000048513897"
-               iyy="0.00093640099"
-               iyz="0.000061136258"
-               izz="0.00055404990" />
+            <origin xyz="-4.5912860e-02  1.0379104e-02 -1.0247188e-01" rpy="0 0 0" />
+            <mass value="2.3801256e-01" />
+            <inertia
+               ixx="4.8440533e-04"
+               ixy="-5.0691989e-06"
+               ixz="-2.7639482e-05"
+               iyy="6.8931084e-04"
+               iyz="7.8890230e-05"
+               izz="3.3000424e-04" />
          </inertial>
       </link>
@@ -601,13 +601,13 @@
          </collision>
          <inertial>
-            <origin xyz="-0.0082599999 0.000056545792 0.0070971896" rpy="0 0 0" />
-            <mass value="0.0060222456" />
-            <inertia
-               ixx="0.00000061965192"
-               ixy="-0.0000000028127992"
-               ixz="0.00000024238121"
-               iyy="0.0000012235266"
-               iyz="0.0000000024168250"
-               izz="0.00000069500159" />
+            <origin xyz="-8.6845430e-03  3.1215919e-04  6.2417800e-03" rpy="0 0 0" />
+            <mass value="3.4935532e-03" />
+            <inertia
+               ixx="3.1731774e-07"
+               ixy="-9.4708822e-09"
+               ixz="1.3547192e-07"
+               iyy="7.0503093e-07"
+               iyz="6.8069408e-09"
+               izz="4.0910623e-07" />
          </inertial>
       </link>

Commit message: Refined joint origin positions in a2 leader

File: ffw_description/urdf/common/leader/ffw_mini_leader_body.urdf.xacro (robot description, xacro)
@@ -41,5 +41,5 @@
          <parent link="${prefix}arm_base_link" />
          <child link="${prefix}arm_l_link1" />
-         <origin xyz="0 0.13070 0" rpy="0 0 0" />
+         <origin xyz="-0.0001 0.13070 0" rpy="0 0 0" />
          <axis xyz="0 1 0" />
          <limit velocity="4.8" effort="1000" lower="-6.28" upper="6.28" />
@@ -149,5 +149,5 @@
          <parent link="${prefix}arm_l_link3" />
          <child link="${prefix}arm_l_link4" />
-         <origin xyz="0.01642 0 -0.04151" rpy="0 0 0" />
+         <origin xyz="0.0165165 0 -0.0415144" rpy="0 0 0" />
          <axis xyz="0 1 0" />
          <limit velocity="4.8" effort="1000" lower="-6.28" upper="6.28" />
@@ -185,5 +185,5 @@
          <parent link="${prefix}arm_l_link4" />
          <child link="${prefix}arm_l_link5" />
-         <origin xyz="-0.01642 0 -0.07802" rpy="0 0 0" />
+         <origin xyz="-0.0165165 0 -0.0780165" rpy="0 0 0" />
          <axis xyz="0 0 1" />
          <limit velocity="4.8" effort="1000" lower="-6.28" upper="6.28" />
@@ -291,5 +291,5 @@
       </link>
       <joint name="${prefix}gripper_l_joint1" type="revolute">
-         <origin xyz="-0.0717 0 -0.137526" rpy="0 0 0"/>
+         <origin xyz="-0.0691039 0.00015 -0.143265" rpy="0 0 0"/>
          <parent link="${prefix}arm_l_link7"/>
          <axis xyz="0 1 0"/>
@@ -328,5 +328,5 @@
          <parent link="${prefix}arm_base_link" />
          <child link="${prefix}arm_r_link1" />
-         <origin xyz="0 -0.13070 0" rpy="0 0 0" />
+         <origin xyz="-0.0001 -0.13070 0" rpy="0 0 0" />
          <axis xyz="0 1 0" />
          <limit velocity="4.8" effort="1000" lower="-6.28" upper="6.28" />
@@ -436,5 +436,5 @@
          <parent link="${prefix}arm_r_link3" />
          <child link="${prefix}arm_r_link4" />
-         <origin xyz="0.01642 0 -0.04151" rpy="0 0 0" />
+         <origin xyz="0.0165165 0 -0.0415144" rpy="0 0 0" />
          <axis xyz="0 1 0" />
          <limit velocity="4.8" effort="1000" lower="-6.28" upper="6.28" />
@@ -472,5 +472,5 @@
          <parent link="${prefix}arm_r_link4" />
          <child link="${prefix}arm_r_link5" />
-         <origin xyz="-0.01642 0 -0.07802" rpy="0 0 0" />
+         <origin xyz="-0.0165165 0 -0.0780165" rpy="0 0 0" />
          <axis xyz="0 0 1" />
          <limit velocity="4.8" effort="1000" lower="-6.28" upper="6.28" />
@@ -578,5 +578,5 @@
       </link>
       <joint name="${prefix}gripper_r_joint1" type="revolute">
-         <origin xyz="-0.0717 -0.002 -0.137526" rpy="0 0 0"/>
+         <origin xyz="-0.0691039 -0.00015 -0.143265" rpy="0 0 0"/>
          <parent link="${prefix}arm_r_link7"/>
          <axis xyz="0 1 0"/>
