Commit message: Added relpose controller for A1

File: ffw_description/ros2_control/ffw_a1_leader/ffw_a1_leader.ros2_control.xacro (robot description, xacro)
@@ -113,5 +113,13 @@
         <param name="Homing Offset">200</param>
       </gpio>
-      <!-- DXL_ENC Homing Offset shifts Present Position with the same sign in both Drive Modes. -->
+      <gpio name="dxl31">
+        <param name="type">dxl</param>
+        <param name="ID">31</param>
+        <state_interface name="Present Position"/>
+        <param name="Drive Mode">0</param>
+        <param name="Homing Offset">0</param>
+        <param name="Return Delay Time">0</param>
+        <param name="Torque Enable">0</param>
+      </gpio>
       <gpio name="dxl32">
         <param name="type">dxl</param>
@@ -120,13 +128,4 @@
         <param name="Drive Mode">1</param>
         <param name="Homing Offset">1366</param>
-        <param name="Return Delay Time">0</param>
-        <param name="Torque Enable">0</param>
-      </gpio>
-      <gpio name="dxl31">
-        <param name="type">dxl</param>
-        <param name="ID">31</param>
-        <state_interface name="Present Position"/>
-        <param name="Drive Mode">0</param>
-        <param name="Homing Offset">0</param>
         <param name="Return Delay Time">0</param>
         <param name="Torque Enable">0</param>
@@ -198,4 +197,13 @@
         <param name="Homing Offset">-200</param>
       </gpio>
+      <gpio name="dxl1">
+        <param name="type">dxl</param>
+        <param name="ID">1</param>
+        <state_interface name="Present Position"/>
+        <param name="Drive Mode">0</param>
+        <param name="Homing Offset">0</param>
+        <param name="Return Delay Time">0</param>
+        <param name="Torque Enable">0</param>
+      </gpio>
       <gpio name="dxl2">
         <param name="type">dxl</param>
@@ -204,13 +212,4 @@
         <param name="Drive Mode">0</param>
         <param name="Homing Offset">1366</param>
-        <param name="Return Delay Time">0</param>
-        <param name="Torque Enable">0</param>
-      </gpio>
-      <gpio name="dxl1">
-        <param name="type">dxl</param>
-        <param name="ID">1</param>
-        <state_interface name="Present Position"/>
-        <param name="Drive Mode">0</param>
-        <param name="Homing Offset">0</param>
         <param name="Return Delay Time">0</param>
         <param name="Torque Enable">0</param>

File: ffw_description/urdf/ffw_a1_leader/ffw_a1_leader.urdf.xacro (robot description, xacro)
@@ -5,10 +5,141 @@
   <xacro:arg name="mock_sensor_commands" default="false" />
   <xacro:arg name="prefix" default="" />
-  <xacro:include filename="$(find ffw_description)/urdf/common/leader/ffw_leader_body.urdf.xacro" />
   <xacro:include filename="$(find ffw_description)/ros2_control/ffw_a1_leader/ffw_a1_leader.ros2_control.xacro" />
   <link name="$(arg prefix)world"/>
-  <xacro:ffw_leader_body parent="$(arg prefix)world" prefix="$(arg prefix)">
+  <joint name="$(arg prefix)joint" type="prismatic">
+    <parent link="$(arg prefix)world"/>
+    <child link="$(arg prefix)arm_base_link" />
     <origin xyz="0 0 0" rpy="0 0 0" />
-  </xacro:ffw_leader_body>
+    <axis xyz="0 0 1" />
+    <limit velocity="4.8" effort="1000" lower="0.0" upper="0.25" />
+    <dynamics damping="0.1" />
+  </joint>
+  <link name="$(arg prefix)arm_base_link"/>
+  <joint name="$(arg prefix)arm_l_joint1" type="revolute">
+    <parent link="$(arg prefix)arm_base_link" />
+    <child link="$(arg prefix)arm_l_link1" />
+    <origin xyz="0 0.1912 0" rpy="0 0 0" />
+    <axis xyz="1 0 0" />
+    <limit velocity="4.8" effort="1000" lower="-6.28" upper="6.28" />
+    <dynamics damping="0.1" />
+  </joint>
+  <link name="$(arg prefix)arm_l_link1"/>
+  <joint name="$(arg prefix)arm_l_joint2" type="revolute">
+    <parent link="$(arg prefix)arm_l_link1" />
+    <child link="$(arg prefix)arm_l_link2" />
+    <origin xyz="0.120795 0.0795 -0.000151884" rpy="0 0 0" />
+    <axis xyz="0 1 0" />
+    <limit velocity="4.8" effort="1000" lower="-6.28" upper="6.28" />
+    <dynamics damping="0.1" />
+  </joint>
+  <link name="$(arg prefix)arm_l_link2"/>
+  <joint name="$(arg prefix)arm_l_joint3" type="revolute">
+    <parent link="$(arg prefix)arm_l_link2" />
+    <child link="$(arg prefix)arm_l_link3" />
+    <origin xyz="-0.00005 0 -0.2295" rpy="0 0 0" />
+    <axis xyz="0 0 1" />
+    <limit velocity="4.8" effort="1000" lower="-6.28" upper="6.28" />
+    <dynamics damping="0.1" />
+  </joint>
+  <link name="$(arg prefix)arm_l_link3"/>
+  <joint name="$(arg prefix)arm_l_joint4" type="revolute">
+    <parent link="$(arg prefix)arm_l_link3" />
+    <child link="$(arg prefix)arm_l_link4" />
+    <origin xyz="0 0 0" rpy="0 0 0" />
+    <axis xyz="0 1 0" />
+    <limit velocity="4.8" effort="1000" lower="-6.28" upper="6.28" />
+    <dynamics damping="0.1" />
+  </joint>
+  <link name="$(arg prefix)arm_l_link4"/>
+  <joint name="$(arg prefix)arm_l_joint5" type="revolute">
+    <parent link="$(arg prefix)arm_l_link4" />
+    <child link="$(arg prefix)arm_l_link5" />
+    <origin xyz="-0.036 0 -0.21345" rpy="0 0 0" />
+    <axis xyz="0 0 1" />
+    <limit velocity="4.8" effort="1000" lower="-6.28" upper="6.28" />
+    <dynamics damping="0.1" />
+  </joint>
+  <link name="$(arg prefix)arm_l_link5"/>
+  <joint name="$(arg prefix)arm_l_joint6" type="revolute">
+    <parent link="$(arg prefix)arm_l_link5" />
+    <child link="$(arg prefix)arm_l_link6" />
+    <origin xyz="0 0 0" rpy="0 0 0" />
+    <axis xyz="0 1 0" />
+    <limit velocity="4.8" effort="1000" lower="-6.28" upper="6.28" />
+    <dynamics damping="0.1" />
+  </joint>
+  <link name="$(arg prefix)arm_l_link6"/>
+  <joint name="$(arg prefix)arm_l_joint7" type="revolute">
+    <parent link="$(arg prefix)arm_l_link6" />
+    <child link="$(arg prefix)arm_l_link7" />
+    <origin xyz="0.0796388 -0.07945 0.0001" rpy="0 0 0" />
+    <axis xyz="1 0 0" />
+    <limit velocity="4.8" effort="1000" lower="-6.28" upper="6.28" />
+    <dynamics damping="0.1" />
+  </joint>
+  <link name="$(arg prefix)arm_l_link7"/>
+  <joint name="$(arg prefix)arm_r_joint1" type="revolute">
+    <parent link="$(arg prefix)arm_base_link" />
+    <child link="$(arg prefix)arm_r_link1" />
+    <origin xyz="0 -0.1912 0" rpy="0 0 0" />
+    <axis xyz="1 0 0" />
+    <limit velocity="4.8" effort="1000" lower="-6.28" upper="6.28" />
+    <dynamics damping="0.1" />
+  </joint>
+  <link name="$(arg prefix)arm_r_link1"/>
+  <joint name="$(arg prefix)arm_r_joint2" type="revolute">
+    <parent link="$(arg prefix)arm_r_link1" />
+    <child link="$(arg prefix)arm_r_link2" />
+    <origin xyz="0.120795198 -0.0795 -0.000251884" rpy="0 0 0" />
+    <axis xyz="0 1 0" />
+    <limit velocity="4.8" effort="1000" lower="-6.28" upper="6.28" />
+    <dynamics damping="0.1" />
+  </joint>
+  <link name="$(arg prefix)arm_r_link2"/>
+  <joint name="$(arg prefix)arm_r_joint3" type="revolute">
+    <parent link="$(arg prefix)arm_r_link2" />
+    <child link="$(arg prefix)arm_r_link3" />
+    <origin xyz="-0.00005 0 -0.2295" rpy="0 0 0" />
+    <axis xyz="0 0 1" />
+    <limit velocity="4.8" effort="1000" lower="-6.28" upper="6.28" />
+    <dynamics damping="0.1" />
+  </joint>
+  <link name="$(arg prefix)arm_r_link3"/>
+  <joint name="$(arg prefix)arm_r_joint4" type="revolute">
+    <parent link="$(arg prefix)arm_r_link3" />
+    <child link="$(arg prefix)arm_r_link4" />
+    <origin xyz="0 0 0" rpy="0 0 0" />
+    <axis xyz="0 1 0" />
+    <limit velocity="4.8" effort="1000" lower="-6.28" upper="6.28" />
+    <dynamics damping="0.1" />
+  </joint>
+  <link name="$(arg prefix)arm_r_link4"/>
+  <joint name="$(arg prefix)arm_r_joint5" type="revolute">
+    <parent link="$(arg prefix)arm_r_link4" />
+    <child link="$(arg prefix)arm_r_link5" />
+    <origin xyz="-0.036 0 -0.21355" rpy="0 0 0" />
+    <axis xyz="0 0 1" />
+    <limit velocity="4.8" effort="1000" lower="-6.28" upper="6.28" />
+    <dynamics damping="0.1" />
+  </joint>
+  <link name="$(arg prefix)arm_r_link5"/>
+  <joint name="$(arg prefix)arm_r_joint6" type="revolute">
+    <parent link="$(arg prefix)arm_r_link5" />
+    <child link="$(arg prefix)arm_r_link6" />
+    <origin xyz="0 0 0" rpy="0 0 0" />
+    <axis xyz="0 1 0" />
+    <limit velocity="4.8" effort="1000" lower="-6.28" upper="6.28" />
+    <dynamics damping="0.1" />
+  </joint>
+  <link name="$(arg prefix)arm_r_link6"/>
+  <joint name="$(arg prefix)arm_r_joint7" type="revolute">
+    <parent link="$(arg prefix)arm_r_link6" />
+    <child link="$(arg prefix)arm_r_link7" />
+    <origin xyz="0.0796388 0.07945 0" rpy="0 0 0" />
+    <axis xyz="1 0 0" />
+    <limit velocity="4.8" effort="1000" lower="-6.28" upper="6.28" />
+    <dynamics damping="0.1" />
+  </joint>
+  <link name="$(arg prefix)arm_r_link7"/>
   <joint name="$(arg prefix)gripper_l_joint1" type="revolute">
     <origin xyz="0 0 0" rpy="0 0 0"/>
@@ -27,4 +158,17 @@
   </joint>
   <link name="$(arg prefix)gripper_r_link1"/>
+  <!-- Until TCP calibration, each tool frame coincides with its seventh arm link. -->
+  <joint name="$(arg prefix)end_effector_l_joint" type="fixed">
+    <parent link="$(arg prefix)arm_l_link7" />
+    <child link="$(arg prefix)end_effector_l_link" />
+    <origin xyz="0 0 0" rpy="0 0 0" />
+  </joint>
+  <link name="$(arg prefix)end_effector_l_link" />
+  <joint name="$(arg prefix)end_effector_r_joint" type="fixed">
+    <parent link="$(arg prefix)arm_r_link7" />
+    <child link="$(arg prefix)end_effector_r_link" />
+    <origin xyz="0 0 0" rpy="0 0 0" />
+  </joint>
+  <link name="$(arg prefix)end_effector_r_link" />
   <xacro:ffw_a1_leader_system
       use_sim="$(arg use_sim)"
