Commit message: Added cartesian pose reference scaling

File: ffw_description/urdf/ffw_a1_leader/ffw_a1_leader.urdf.xacro (robot description, xacro)
@@ -162,5 +162,5 @@
     <parent link="$(arg prefix)arm_l_link7" />
     <child link="$(arg prefix)end_effector_l_link" />
-    <origin xyz="0 0 0" rpy="0 0 0" />
+    <origin xyz="0 0 -0.15" rpy="0 0 0" />
   </joint>
   <link name="$(arg prefix)end_effector_l_link" />
@@ -168,5 +168,5 @@
     <parent link="$(arg prefix)arm_r_link7" />
     <child link="$(arg prefix)end_effector_r_link" />
-    <origin xyz="0 0 0" rpy="0 0 0" />
+    <origin xyz="0 0 -0.15" rpy="0 0 0" />
   </joint>
   <link name="$(arg prefix)end_effector_r_link" />
